File: Hardware/Main_PCB/Floor.kicad_sch (KiCad schematic)
At the start: 14 parts, among them J1 Capacitive Soil Moisture, J10 Capacitive Soil Moisture, J11 Capacitive Soil Moisture, J12 Capacitive Soil Moisture, J13 Capacitive Soil Moisture, J14 Capacitive Soil Moisture, J3 Magnetic THT Pins Male, J4 Magnetic THT Pins Male, J8 Capacitive Soil Moisture, J9 Capacitive Soil Moisture, U1 WS2811, U5 WS2811, U6 WS2811, U7 WS2811

Commit message: Updated schematic
Parts:
- renumbered J3 to J17, J4 to J18, J14 to J19, J13 to J20, J12 to J21, J11 to J22, J10 to J23, J9 to J24, J8 to J25, J1 to J26, U1 to U16, U5 to U17, U6 to U18, U7 to U19
Changed lines of the file:
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@@
 		(dnp no)
 		(fields_autoplaced yes)
-		(property "Reference" "J3"
+		(property "Reference" "J17"
 			(at 36.83 95.2499 0)
 			(show_name no)
@@
 		(instances
 			(project "GrowHub_Elec"
-				(path "/af001b7e-1c5e-4b7a-a0b4-e6af7dd78ca9/c7e8d3f4-060b-4d22-8783-e9f4f221b151"
-					(reference "J3")
+				(path "/af001b7e-1c5e-4b7a-a0b4-e6af7dd78ca9/60e449cd-fd6d-4899-8c59-5b83fe162284"
+					(reference "J17")
 					(unit 1)
 				)
@@
 		(dnp no)
 		(fields_autoplaced yes)
-		(property "Reference" "J4"
+		(property "Reference" "J18"
 			(at 36.83 139.6999 0)
 			(show_name no)
@@
 		(instances
 			(project "GrowHub_Elec"
-				(path "/af001b7e-1c5e-4b7a-a0b4-e6af7dd78ca9/c7e8d3f4-060b-4d22-8783-e9f4f221b151"
-					(reference "J4")
+				(path "/af001b7e-1c5e-4b7a-a0b4-e6af7dd78ca9/60e449cd-fd6d-4899-8c59-5b83fe162284"
+					(reference "J18")
 					(unit 1)
 				)
@@
 		(dnp no)
 		(fields_autoplaced yes)
-		(property "Reference" "U5"
+		(property "Reference" "U17"
 			(at 146.9233 91.44 0)
 			(show_name no)
@@
 		(instances
 			(project "GrowHub_Elec"
-				(path "/af001b7e-1c5e-4b7a-a0b4-e6af7dd78ca9/c7e8d3f4-060b-4d22-8783-e9f4f221b151"
-					(reference "U5")
+				(path "/af001b7e-1c5e-4b7a-a0b4-e6af7dd78ca9/60e449cd-fd6d-4899-8c59-5b83fe162284"
+					(reference "U17")
 					(unit 1)
 				)
@@
 		(dnp no)
 		(fields_autoplaced yes)
-		(property "Reference" "J10"
+		(property "Reference" "J23"
 			(at 177.165 118.11 0)
 			(show_name no)
@@
 		(instances
 			(project "GrowHub_Elec"
-				(path "/af001b7e-1c5e-4b7a-a0b4-e6af7dd78ca9/c7e8d3f4-060b-4d22-8783-e9f4f221b151"
-					(reference "J10")
+				(path "/af001b7e-1c5e-4b7a-a0b4-e6af7dd78ca9/60e449cd-fd6d-4899-8c59-5b83fe162284"
+					(reference "J23")
 					(unit 1)
 				)
@@
 		(dnp no)
 		(fields_autoplaced yes)
-		(property "Reference" "U1"
+		(property "Reference" "U16"
 			(at 145.6533 69.85 0)
 			(show_name no)
@@
 		(instances
 			(project "GrowHub_Elec"
-				(path "/af001b7e-1c5e-4b7a-a0b4-e6af7dd78ca9/c7e8d3f4-060b-4d22-8783-e9f4f221b151"
-					(reference "U1")
+				(path "/af001b7e-1c5e-4b7a-a0b4-e6af7dd78ca9/60e449cd-fd6d-4899-8c59-5b83fe162284"
+					(reference "U16")
 					(unit 1)
 				)
@@
 		(dnp no)
 		(fields_autoplaced yes)
-		(property "Reference" "U7"
+		(property "Reference" "U19"
 			(at 146.9233 132.08 0)
 			(show_name no)
@@
 		(instances
 			(project "GrowHub_Elec"
-				(path "/af001b7e-1c5e-4b7a-a0b4-e6af7dd78ca9/c7e8d3f4-060b-4d22-8783-e9f4f221b151"
-					(reference "U7")
+				(path "/af001b7e-1c5e-4b7a-a0b4-e6af7dd78ca9/60e449cd-fd6d-4899-8c59-5b83fe162284"
+					(reference "U19")
 					(unit 1)
 				)
@@
 		(dnp no)
 		(fields_autoplaced yes)
-		(property "Reference" "J9"
+		(property "Reference" "J24"
 			(at 177.165 133.35 0)
 			(show_name no)
@@
 		(instances
 			(project "GrowHub_Elec"
-				(path "/af001b7e-1c5e-4b7a-a0b4-e6af7dd78ca9/c7e8d3f4-060b-4d22-8783-e9f4f221b151"
-					(reference "J9")
+				(path "/af001b7e-1c5e-4b7a-a0b4-e6af7dd78ca9/60e449cd-fd6d-4899-8c59-5b83fe162284"
+					(reference "J24")
 					(unit 1)
 				)
@@
 		(dnp no)
 		(fields_autoplaced yes)
-		(property "Reference" "J8"
+		(property "Reference" "J25"
 			(at 177.165 147.32 0)
 			(show_name no)
@@
 		(instances
 			(project "GrowHub_Elec"
-				(path "/af001b7e-1c5e-4b7a-a0b4-e6af7dd78ca9/c7e8d3f4-060b-4d22-8783-e9f4f221b151"
-					(reference "J8")
+				(path "/af001b7e-1c5e-4b7a-a0b4-e6af7dd78ca9/60e449cd-fd6d-4899-8c59-5b83fe162284"
+					(reference "J25")
 					(unit 1)
 				)
@@
 		(dnp no)
 		(fields_autoplaced yes)
-		(property "Reference" "U6"
+		(property "Reference" "U18"
 			(at 146.9233 113.03 0)
 			(show_name no)
@@
 		(instances
 			(project "GrowHub_Elec"
-				(path "/af001b7e-1c5e-4b7a-a0b4-e6af7dd78ca9/c7e8d3f4-060b-4d22-8783-e9f4f221b151"
-					(reference "U6")
+				(path "/af001b7e-1c5e-4b7a-a0b4-e6af7dd78ca9/60e449cd-fd6d-4899-8c59-5b83fe162284"
+					(reference "U18")
 					(unit 1)
 				)
@@
 		(dnp no)
 		(fields_autoplaced yes)
-		(property "Reference" "J14"
+		(property "Reference" "J19"
 			(at 177.165 60.96 0)
 			(show_name no)
@@
 		(instances
 			(project "GrowHub_Elec"
-				(path "/af001b7e-1c5e-4b7a-a0b4-e6af7dd78ca9/c7e8d3f4-060b-4d22-8783-e9f4f221b151"
-					(reference "J14")
+				(path "/af001b7e-1c5e-4b7a-a0b4-e6af7dd78ca9/60e449cd-fd6d-4899-8c59-5b83fe162284"
+					(reference "J19")
 					(unit 1)
 				)
@@
 		(dnp no)
 		(fields_autoplaced yes)
-		(property "Reference" "J13"
+		(property "Reference" "J20"
 			(at 177.165 74.93 0)
 			(show_name no)
@@
 		(instances
 			(project "GrowHub_Elec"
-				(path "/af001b7e-1c5e-4b7a-a0b4-e6af7dd78ca9/c7e8d3f4-060b-4d22-8783-e9f4f221b151"
-					(reference "J13")
+				(path "/af001b7e-1c5e-4b7a-a0b4-e6af7dd78ca9/60e449cd-fd6d-4899-8c59-5b83fe162284"
+					(reference "J20")
 					(unit 1)
 				)
@@
 		(dnp no)
 		(fields_autoplaced yes)
-		(property "Reference" "J12"
+		(property "Reference" "J21"
 			(at 177.165 87.63 0)
 			(show_name no)
@@
 		(instances
 			(project "GrowHub_Elec"
-				(path "/af001b7e-1c5e-4b7a-a0b4-e6af7dd78ca9/c7e8d3f4-060b-4d22-8783-e9f4f221b151"
-					(reference "J12")
+				(path "/af001b7e-1c5e-4b7a-a0b4-e6af7dd78ca9/60e449cd-fd6d-4899-8c59-5b83fe162284"
+					(reference "J21")
 					(unit 1)
 				)
@@
 		(dnp no)
 		(fields_autoplaced yes)
-		(property "Reference" "J1"
+		(property "Reference" "J26"
 			(at 177.165 161.29 0)
 			(show_name no)
@@
 		(instances
 			(project "GrowHub_Elec"
-				(path "/af001b7e-1c5e-4b7a-a0b4-e6af7dd78ca9/c7e8d3f4-060b-4d22-8783-e9f4f221b151"
-					(reference "J1")
+				(path "/af001b7e-1c5e-4b7a-a0b4-e6af7dd78ca9/60e449cd-fd6d-4899-8c59-5b83fe162284"
+					(reference "J26")
 					(unit 1)
 				)
@@
 		(dnp no)
 		(fields_autoplaced yes)
-		(property "Reference" "J11"
+		(property "Reference" "J22"
 			(at 177.165 102.87 0)
 			(show_name no)
@@
 		(instances
 			(project "GrowHub_Elec"
-				(path "/af001b7e-1c5e-4b7a-a0b4-e6af7dd78ca9/c7e8d3f4-060b-4d22-8783-e9f4f221b151"
-					(reference "J11")
-					(unit 1)
-				)
+				(path "/af001b7e-1c5e-4b7a-a0b4-e6af7dd78ca9/60e449cd-fd6d-4899-8c59-5b83fe162284"
+					(reference "J22")
+					(unit 1)
+				)

Commit message: Hardware Week 2
Parts:
- added U17: ADG706BRU, ADG706BRU:SOP65P640X120-28N, symbol ADG706BRU:ADG706BRU
- added U18: ADS1115IDGSR, ADS1115IDGSR:SOP50P490X110-10N, symbol ADS1115IDGSR:ADS1115IDGSR
- added U19: PCA9685BS_118, PCA9685BS_118:QFN65P600X600X100-29N, symbol PCA9685BS_118:PCA9685BS_118
- added U20: MCP23017T-E_SO, MCP23017T-E_SO:SOIC127P1030X265-28N, symbol MCP23017T-E_SO:MCP23017T-E_SO
- added U21: P82B96D, P82B96D:SOIC127P599X175-8N, symbol P82B96D:P82B96D
- added U22: DS28E07Q_T, DS28E07Q_T:SON95P300X300X80-7N, symbol DS28E07Q_T:DS28E07Q_T
- renumbered J26 to J1, J23 to J10, J22 to J11, J21 to J12, J20 to J13, J19 to J14, J17 to J3, J18 to J4, J25 to J8, J24 to J9, U16 to U1, U17 to U5, U18 to U6, U19 to U7
Other:
- moved on the sheet: J1, J10, J11, J12, J13, J14, J3, J4, J8, J9, U1, U5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

Commit message: schematic newest
Parts:
- removed J3, J4: Magnetic THT Pins Male, symbol Connector:DA15_Socket_MountingHoles
- added C25, C26, C27, C28, C55, C57, C65: 1uF, symbol Device:C
- added C53: 10uF, symbol Device:C
- added C54, C56, C58, C66: 100nF, symbol Device:C
- added C59, C60: 10nF, symbol Device:C
- added J7: Molex Micro-Fit 3.0, 0430451213, symbol 0430451213:0430451213
- added R1, R6: 1K, symbol Device:R
- added R3, R4, R5, R7: 10K, symbol Device:R
- added U12: AS7341-DLGM, AS7341-DLGM:XDCR_AS7341-DLGM, symbol AS7341-DLGM:AS7341-DLGM
- added U16, U23: TPS7A2033PDQNR, TPS7A2033PDQNR:VREG_TPS7A2033PDQNR, symbol TPS7A2033PDQNR:TPS7A2033PDQNR
Connections:
- net GND: now reaches U18.1 (ADDR)
- net GND: now also U17.12 (GND), U17.27 (VSS), U18.3 (GND), U19.1 (A3), U19.2 (A4), U19.21 (A5), U19.22 (EXTCLK), U19.26 (A0), U19.27 (A1), U19.28 (A2), U20.15 (A0), U20.16 (A1), U20.17 (A2), C25.2, C26.2, C27.2, C28.2, C53.2, C54.2, C55.2, C56.2, C57.2, C58.2, C59.2, C60.2, C65.2, C66.2, J7.7 (7_GND), J7.8 (8_GND), R4.1, U16.2 (GND), U16.5 (EXP), U23.2 (GND), U23.5 (EXP)
- net Ain_0: now reaches U18.4 (AIN0)
- net Ain_0: now also C60.1, R6.1
- net at U18.5 (AIN1): now also C59.1, R1.2
- net at U18.6 (AIN2): now also R3.1, R4.2
- net +3V3: now reaches U18.8 (VDD)
- net +3V3: now also U17.18 (EN), U19.25 (VDD), C57.1, C58.1, C65.1, C66.1, R7.1
- net OE: now reaches U19.20 (~{OE})
- net OE: now also R7.2
- net SCL_1: now reaches U19.23 (SCL)
- net SDA_1: now reaches U19.24 (SDA)
- net SCL_0: now reaches U20.12 (SCK)
- net SDA_0: now reaches U20.13 (SDA)
- net Probe_rail_EN: now reaches U20.21 (GPA0)
- net Probe_rail_EN: now also U16.3 (EN)
- net ADC_MUX_0: now reaches U20.22 (GPA1)
- net ADC_MUX_0: now also U17.17 (A0)
- net ADC_MUX_1: now reaches U20.23 (GPA2)
- net ADC_MUX_1: now also U17.16 (A1)
- net ADC_MUX_2: now reaches U20.24 (GPA3)
- net ADC_MUX_2: now also U17.15 (A2)
- net ADC_MUX_3: now reaches U20.25 (GPA4)
- net ADC_MUX_3: now also U17.14 (A3)
- net at U17.1 (VDD): now also C55.1, C56.1, R5.2
- net ID_1: now reaches U17.10 (S10)
- net ID_0: now reaches U17.11 (S9)
- net Soil_0: now reaches U17.19 (S1)
- net Soil_1: now reaches U17.20 (S2)
- net Soil_2: now reaches U17.21 (S3)
- net Soil_3: now reaches U17.22 (S4)
- net Soil_4: now reaches U17.23 (S5)
- net Soil_5: now reaches U17.24 (S6)
- net Soil_6: now reaches U17.25 (S7)
- net Soil_7: now reaches U17.26 (S8)
- net at U17.28 (D): now also R6.2
- net ID_7: now reaches U17.4 (S16)
- net ID_6: now reaches U17.5 (S15)
- net ID_5: now reaches U17.6 (S14)
- net ID_4: now reaches U17.7 (S13)
- net ID_3: now reaches U17.8 (S12)
- net ID_2: now reaches U17.9 (S11)
- new net: C28.1, U16.1 (OUT)
- new net: C53.1, C54.1, J7.10 (10_5V), J7.9 (9_5V)
- new net +5V: C26.1, C27.1, R3.2, R5.1, U16.4 (IN), U23.3 (EN), U23.4 (IN)
- new net TPS7A20_Vout: C25.1, U23.1 (OUT)
- new net VCC_SW: R1.1
- no-connect marks 0 -> 2
Other:
- note added: "I need MOSFET for LEDs"
- note added: "Logic LDO"
- note added: "Might get deferred if we include hydroponics"
- note added: "Probe-Rail LDO"

Commit message: Week 4 Schematic
Parts:
- removed J1, J10, J11, J12, J13, J14, J8, J9: Capacitive Soil Moisture, symbol Connector:Conn_01x03_Socket
- removed R1: 1K, symbol Device:R
- removed R3, R4: 10K, symbol Device:R
- removed U1, U5, U6, U7: WS2811, symbol Driver_LED:WS2811
- added C10, C69, C70, C74, C77, C78, C79, C80, C81: 100nF, symbol Device:C
- added C3, C75: 220uF, symbol Device:C_Polarized
- added C64, C84: 10nF, symbol Device:C
- added C68: 220uF, symbol Device:C
- added C73, C76: 1uF, symbol Device:C
- added D19, D20, D27, D28, D6, D9: ESD5Zxx, Diode_SMD:D_SOD-523, symbol Diode:ESD5Zxx
- added D21, D22, D23, D24: SS25, Diode_SMD:D_SMA, symbol Diode:SS25
- added D29, D30, D31: SS16, Diode_SMD:D_SMA, symbol Diode:SS16
- added J3, J4, J6, J8: B2B-PH-K-S, B2B-PH-K-S:JST_B2B-PH-K-S, symbol B2B-PH-K-S:B2B-PH-K-S
- added Q15, Q7: BSS138BK-215, TL431CDBZR215, symbol BSS138BK-215:BSS138BK-215
- added Q17, Q26, Q27, Q3, Q4, Q5, Q6: AO3422, SOT95P237X112-3N, symbol AO3422:AO3422
- added R102, R103, R104, R105, R106, R107, R108, R109, R125, R14, R88: 1K, symbol Device:R
- added R110, R114, R116, R118, R126, R68, R70, R73, R94: 100K, symbol Device:R
- added R111, R127: 10K, symbol Device:R
- added R112: 1M, symbol Device:R
- added R113, R115, R117: 100, symbol Device:R
- added R128: 47K, symbol Device:R
- added R62, R63: 0, symbol Device:R
- added R64, R65: R_X, symbol Device:R
- added R67, R69, R71, R74: 33, symbol Device:R
- added R8, R9: 4.7K, symbol Device:R
- added U3: SHT4XI-DIGITAL, SHT4XI-DIGITAL:SHT4XI-DIGITAL, symbol SHT4XI-DIGITAL:SHT4XI-DIGITAL
- R5: value 10K -> 10
Connections:
- net OE is gone; now on net OE_X: R7.2, U19.20 (~{OE})
- net SCL_0 is gone; now on net SCL_X: U20.12 (SCK)
- net SCL_1 is gone; now on net SCL_X: U19.23 (SCL)
- net SDA_0 is gone; now on net SDA_X: U20.13 (SDA)
- net SDA_1 is gone; now on net SDA_X: U19.24 (SDA)
- net TPS7A20_Vout is gone; now on net +3V3: C25.1, U23.1 (OUT)
- net +3V3: now also C28.1, U12.1 (VDD), U16.1 (OUT), U20.9 (VDD), C10.2, C78.1, Q7.1 (G), R8.2, R9.2, U3.3 (VDD); no longer U17.18 (EN)
- net +5V: now also U21.8 (VCC), C70.1, R64.2, R65.2
- net ADC_MUX_0: now also U20.1 (GPB0); no longer U20.22 (GPA1)
- net ADC_MUX_1: now also U20.2 (GPB1); no longer U20.23 (GPA2)
- net ADC_MUX_2: now also U20.3 (GPB2); no longer U20.24 (GPA3)
- net ADC_MUX_3: now also U20.4 (GPB3); no longer U20.25 (GPA4)
- net Ain_0: no longer U18.4 (AIN0)
- net GND: now also U12.3 (GND), U12.5 (PGND), U19.11 (VSS), U19.29 (EXP), U20.10 (VSS), U21.4 (GND), U22.3 (GND), U22.7 (EP), C10.1, C3.2, C64.2, C68.2, C69.2, C70.2, C73.1, C74.2, C75.2, C76.1, C77.2, C78.2, C79.2, C80.2, C81.2, C84.2, D19.2 (A), D20.2 (A), D27.2 (A), D28.2 (A), D6.2 (A), D9.2 (A), Q17.2 (S), Q26.2 (S), Q27.2 (S), Q3.2 (S), Q4.2 (S), R110.1, R114.1, R116.1, R118.1, R127.1, R128.2, R68.2, R70.2, U3.4 (VSS)
- net Probe_rail_EN: now also U20.6 (GPB5); no longer U16.3 (EN), U20.21 (GPA0)
- net Soil_0: now also R14.2; no longer U17.19 (S1)
- net Soil_1: now also R102.2; no longer U17.20 (S2)
- net Soil_2: now also R103.2; no longer U17.21 (S3)
- net Soil_3: now also R104.2; no longer U17.22 (S4)
- net Soil_4: now also R105.2; no longer U17.23 (S5)
- net Soil_5: now also R106.2; no longer U17.24 (S6)
- net Soil_6: now also R107.2; no longer U17.25 (S7)
- net Soil_7: now also R108.2; no longer U17.26 (S8)
- net TRAY_EXC: now reaches U19.19 (LED15)
- net TRAY_EXC: now also U20.8 (GPB7), R111.1
- net CH1: now reaches U19.3 (LED0)
- net CH1: now also R67.1
- net CH2: now reaches U19.4 (LED1)
- net CH2: now also R69.1
- net CH3: now reaches U19.5 (LED2)
- net CH3: now also R71.1
- net CH4: now reaches U19.6 (LED3)
- net CH4: now also R74.1
- net OE_X: now reaches J7.1
- net OE_X: now also D9.1 (K)
- net at C53.1, C54.1, J7.10 (10_5V)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: now also C68.1
- net 1-Wire_X: now reaches J7.11
- net 1-Wire_X: now also U22.2 (IO), D20.1 (K)
- net nRESET_X: now reaches J7.2
- net nRESET_X: now also C59.1, U16.3 (EN), U20.18 (~{RESET}), C69.1, R128.1, R88.2
- net SCL_F0: now reaches J7.3
- net SDA_F0: now reaches J7.4
- net VALVE_RAIL: now reaches J7.5
- net VALVE_RAIL: now also C79.1, C80.1, C81.1, D29.1 (K), D30.1 (K), D31.1 (K), J4.1, J6.1, J8.1
- net SCL_X: now reaches U12.2 (SCL)
- net SCL_X: now also U18.10 (SCL), U21.7 (SY), R63.1, R8.1, U3.2 (SCL)
- net SDA_X: now reaches U12.8 (SDA)
- net SDA_X: now also U18.9 (SDA), U21.1 (SX), R62.1, R9.1, U3.1 (SDA)
- net at U18.5 (AIN1): no longer C59.1
- net SD_X: now reaches U21.2 (RX)
- net SD_X: now also U21.3 (TX), D6.1 (K), R62.2, R64.1
- net SC_X: now reaches U21.5 (TY)
- net SC_X: now also U21.6 (RY), D19.1 (K), R63.2, R65.1
- net at U18.7 (AIN3): now also C64.1, R109.1
- net Valve_5: now reaches U20.26 (GPA5)
- net Valve_6: now reaches U20.27 (GPA6)
- net Valve_7: now reaches U20.28 (GPA7)
- net AM_EN: now reaches U20.5 (GPB4)
- net AM_EN: now also U17.18 (EN)
- new net: D27.1 (K), J3.2, R109.2, R110.2
- new net: C84.1, R125.1, U18.4 (AIN0)
- new net: D31.2 (A), J8.2, Q27.3 (D)
- new net: R125.2, R126.1, R127.2
- new net: D29.2 (A), J4.2, Q17.3 (D)
- new net: Q5.1 (G), R71.2, R73.1
- new net: R14.1, U17.19 (S1)
- new net: D28.1 (K), J3.1, R111.2
- new net: Q3.1 (G), R67.2, R68.1
- new net: D30.2 (A), J6.2, Q26.3 (D)
- new net: Q27.1 (G), R117.2, R118.2
- new net: Q4.1 (G), R69.2, R70.1
- new net: Q17.1 (G), R113.2, R114.2
- new net: D24.2 (A), Q6.3 (D)
- new net: Q26.1 (G), R115.2, R116.2
- new net: R102.1, U17.20 (S2)
- new net: R103.1, U17.21 (S3)
- new net: R104.1, U17.22 (S4)
- new net: R105.1, U17.23 (S5)
- new net: R106.1, U17.24 (S6)
- new net: R107.1, U17.25 (S7)
- new net: R108.1, U17.26 (S8)
- new net: D23.2 (A), Q5.3 (D)
- new net: J3., R112.1
- new net: J3., R112.2
- new net: Q6.1 (G), R74.2, R94.1
- new net +24V: C3.1, C73.2, C74.1, C75.1, C76.2, C77.1, D21.1 (K), D22.1 (K), D23.1 (K), D24.1 (K), R126.2
- new net R_LED-: D22.2 (A), Q4.3 (D)
- new net Valve_0: R113.1, U20.21 (GPA0)
- new net Valve_1: R115.1, U20.22 (GPA1)
- new net Valve_2: R117.1, U20.23 (GPA2)
- new net Valve_3: U20.24 (GPA3)
- new net Valve_4: U20.25 (GPA4)
- new net W_LED-: D21.2 (A), Q3.3 (D)
- new net X_LED-: Q5.2 (S), Q6.2 (S), R73.2, R94.2
- no-connect marks 2 -> 22
Other:
- note added: "Buffered option - Without R62/R63 Plain I2C includes them"
- note added: "CH3/CH4 are RESERVED"
- note added: "Floor LDO"
- note added: "For future versions"
- note added: "Lowered amount of Valve FETs made it unreliant"
- note added: "Might not be needed bead"
- note added: "Needs Pogo pin peripheral work depending which design i choose"
- note added: "Not on the PCB"
- note added: "Tray electrodes"
- note added: "Usable LED strips"
- note added: "Valve Driver"
- note removed: "I need MOSFET for LEDs"
- moved on the sheet: C25, C26, C27, C28, C53, C54, C55, C56, C57, C58, C60, J7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
