File: Hardware/Main_PCB/GrowHub_Elec.kicad_sch (KiCad schematic)
At the start: 7 parts, among them IC1 74AHCT125D,118, J2 Magnetic THT Pins Female, J5 Magnetic THT Pins Female, U2 SCD41-D-R2, U3 SHT4XI-DIGITAL, U4 VEML7700-TT, X1 ESP32-S3-WROOM-1-N16R8

Commit message: Week 1 Schematics
Parts:
- added IC2: LMR33610BDDAR, LMR33610BDDAR:LMR33610BDDAR, symbol LMR33610BDDAR:LMR33610BDDAR
- added U10, U11, U8, U9: TCA9548APWR, TCA9548APWR:SOP65P640X120-24N, symbol TCA9548APWR:TCA9548APWR
- added U12: NAU7802SGI, NAU7802SGI:SOIC127P600X175-16N, symbol NAU7802SGI:NAU7802SGI
- added U13: INA226AIDGSR, INA226AIDGSR:SOP50P490X110-10N, symbol INA226AIDGSR:INA226AIDGSR
- added U14: LMR33630ADDA, LMR33630ADDA:VREG_LM5017MR_NOPB, symbol LMR33630ADDA:LMR33630ADDA
- added U15: LTC4364IS-2_PBF, LTC4364IS-2_PBF:SO-16_S, symbol LTC4364IS-2_PBF:LTC4364IS-2_PBF
Connections:
- no-connect marks 0 -> 2
Other:
- sheet Floor Sheet renamed Basic_Floor_PCB
- added sheet Main_Floor_PCB (Main_Floor_PCB.kicad_sch)
- note added: "MCU+passives"
- moved on the sheet: IC1, J2, J5, U2, U3, U4, X1

Commit message: Updated schematic
Parts:
- removed U12: NAU7802SGI, NAU7802SGI:SOIC127P600X175-16N, symbol NAU7802SGI:NAU7802SGI
- removed U8: TCA9548APWR, TCA9548APWR:SOP65P640X120-24N, symbol TCA9548APWR:TCA9548APWR
- removed X1: ESP32-S3-WROOM-1-N16R8, SMD, symbol ESP32-S3-WROOM-1-N16R8:ESP32-S3-WROOM-1-N16R8
- added C1, C17, C18, C19, C20, C25, C26, C27, C28, C9: 22uF, symbol Device:C_Polarized
- added C10, C12, C16, C24, C29, C3, C31, C34, C35: 100nF, symbol Device:C
- added C11, C14, C21: 10uF, symbol Device:C_Polarized
- added C13, C22: 220nF, symbol Device:C
- added C15, C23, C32, C33: 1uF, symbol Device:C_Polarized
- added C2, C5, C6, C8: TBD, symbol Device:C
- added C30: 100uF, symbol Device:C_Polarized
- added C4, C7: 12pF, symbol Device:C
- added J15, J16: JTAG, symbol Connector:Conn_01x04_Pin
- added J6: USB_OTG, symbol Connector:USB_OTG
- added J7: Boot Option, symbol Connector:Conn_01x02_Pin
- added L1, L2: 8uH, 14mΩ, symbol Device:L
- added Q1: FDB3632, FDB3632:TO254P1524X483-3N, symbol FDB3632:FDB3632
- added Q2: FDMS86101, FDMS86252, symbol FDMS86101:FDMS86101
- added R1, R3, R4 (x2), R5, R6, R7: TBD, symbol Device:R
- added R10, R11, R28, R29, R30, R31, R32, R33, R34, R35, R36, R37, R38, R39, R40, R41, R42, R43, R44, R8, R9: 10K, symbol Device:R
- added R12, R13: 2.2K, symbol Device:R
- added R14, R24: 10, symbol Device:R
- added R15, R16, R18, R19, R23: 100K, symbol Device:R
- added R17: 24.9K, symbol Device:R
- added R2, R47, R48, R49: R_45deg, symbol Device:R_45deg
- added R20: 43.3K, symbol Device:R
- added R21: 3.01K, symbol Device:R
- added R22: 6.04K, symbol Device:R
- added R25: 15m, symbol Device:R
- added R26: 110K, symbol Device:R
- added R27: 4.02K, symbol Device:R
- added R45, R46: 47, symbol Device:R
- added SW1: SW_Push, symbol Switch:SW_Push
- added U1: NAU7802SGI, NAU7802SGI:SOIC127P600X175-16N, symbol NAU7802SGI:NAU7802SGI
- added U12: TCA9548APWR, TCA9548APWR:SOP65P640X120-24N, symbol TCA9548APWR:TCA9548APWR
- added U8: ESP32-S3-WROOM-1U-N16R8, ESP32-S3-WROOM-1U-N16R8:XCVR_ESP32-S3-WROOM-1U-N16R8, symbol ESP32-S3-WROOM-1U-N16R8:ESP32-S3-WROOM-1U-N16R8
- added Y1: 32.768KHz, symbol Device:Crystal
- added Z1, Z2: DDZ9702T-7, DDZ9702T7, symbol DDZ9702T-7:DDZ9702T-7
Connections:
- net +24V: now also U13.8 (VBUS), U14.2 (VIN), U14.3 (EN), U15.1 (OUT), U15.8 (VCC), C13.2, C14.1, C30.1, Q1.2, R23.2, R25.1, R26.2
- net +5V: now also IC2.2 (VIN), IC2.3 (EN), U10.24 (VCC), U11.24 (VCC), U13.6 (VS), U9.24 (VCC), C21.1, C22.2, C31.1, R31.1, R32.1, R42.1, R43.1, R44.1, U12.24 (VCC)
- net GND: now also IC2.1 (PGND), IC2.9 (EP), U10.1 (A0), U10.12 (GND), U10.2 (A1), U10.21 (A2), U11.1 (A0), U11.12 (GND), U11.2 (A1), U11.21 (A2), U13.7 (GND), U14.1 (PGND), U14.9 (AGND), U15.12 (GND), U3.4 (VSS), U4.3 (GND), U9.1 (A0), U9.12 (GND), U9.2 (A1), U9.21 (A2), C1.2, C10.1, C11.2, C12.2, C13.1, C14.2, C15.2, C2.1, C20.2, C21.2, C22.1, C23.2, C28.2, C29.2, C3.2, C30.2, C31.2, C32.2, C33.2, C35.2, C4.2, C5.1, C6.1, C7.2, C8.2, C9.2, J16.4 (Pin_4), J6.5 (GND), J7.2 (Pin_2), R17.1, R20.1, R21.1, R27.1, R47.1, R48.1, SW1.1, U1.7 (REFN), U1.8 (AVSS), U1.9 (DVSS), U12.1 (A0), U12.12 (GND), U12.2 (A1), U12.21 (A2), U8.1 (GND), U8.40 (GND), U8.41_1 (GND), U8.41_2 (GND), U8.41_3 (GND), U8.41_4 (GND), U8.41_5 (GND), U8.41_6 (GND), U8.41_7 (GND), U8.41_8 (GND), U8.41_9 (GND)
- net at U13.3 (ALERT): now also R44.2
- net at U13.4 (SDA): now also R42.2
- net at U13.5 (SCL): now also R43.2
- net SDA: now reaches U3.1 (SDA)
- net SDA: now also U2.10 (SDA), U4.4 (SDA), R10.2, R13.2, R9.2
- net SCL: now reaches U3.2 (SCL)
- net SCL: now also U2.9 (SCL), U4.1 (SCL), R11.2, R12.2, R8.2
- net +3V3: now reaches U3.3 (VDD)
- net +3V3: now also U2.19 (VDDH), U2.7 (VDD), C1.1, C10.2, C3.1, C9.1, J16.1 (Pin_1), R1.2, R10.1, R11.1, R12.1, R13.1, R14.2, R28.2, R29.2, R30.2, R33.2, R34.2, R35.2, R36.2, R37.2, R38.2, R39.2, R40.2, R41.2, R8.1, R9.1, U1.15 (DVDD), U8.2 (3V3)
- net TCA9548A SCX: now reaches U9.10 (SD3)
- net TCA9548A SCX: now also U10.10 (SD3), U10.11 (SC3), U10.13 (SD4), U10.15 (SD5), U10.16 (SC5), U10.17 (SD6), U10.18 (SC6), U10.19 (SD7), U10.20 (SC7), U10.4 (SD0), U10.5 (SC0), U10.6 (SD1), U10.7 (SC1), U10.8 (SD2), U10.9 (SC2), U11.10 (SD3), U11.11 (SC3), U11.13 (SD4), U11.15 (SD5), U11.16 (SC5), U11.17 (SD6), U11.18 (SC6), U11.19 (SD7), U11.20 (SC7), U11.4 (SD0), U11.5 (SC0), U11.6 (SD1), U11.7 (SC1), U11.8 (SD2), U11.9 (SC2), U9.11 (SC3), U9.13 (SD4), U9.15 (SD5), U9.16 (SC5), U9.17 (SD6), U9.18 (SC6), U9.19 (SD7), U9.20 (SC7), U9.4 (SD0), U9.5 (SC0), U9.6 (SD1), U9.7 (SC1), U9.8 (SD2), U9.9 (SC2), R31.2, R32.2, U12.10 (SD3), U12.11 (SC3), U12.13 (SD4), U12.15 (SD5), U12.16 (SC5), U12.17 (SD6), U12.18 (SC6), U12.19 (SD7), U12.20 (SC7), U12.4 (SD0), U12.5 (SC0), U12.6 (SD1), U12.7 (SC1), U12.8 (SD2), U12.9 (SC2)
- net at U9.22 (SCL): now also R29.1
- net at U9.23 (SDA): now also R28.1
- net at U9.3 (~{RESET}): now also R30.1
- net at U4.2 (VDD): now also C11.1, C12.1, R14.1
- net at U15.10 (UV): now also R22.2, R23.1
- net at U15.11 (OV): now also R21.2, R22.1
- net at U15.15 (TMR): now also C29.1
- net at U15.16 (FB): now also R26.1, R27.2
- net at U15.2 (SENSE): now also Q2.5 (D_1), R25.2
- net at U15.4 (DGATE): now also Q2.4 (G), Z2.1 (K)
- net at U15.5 (SOURCE): now also Q1.3, Q2.1 (S_1), Z1.2 (A), Z2.2 (A)
- net at U15.6 (HGATE): now also R24.1, Z1.1 (K)
- net PG: now reaches U14.4 (PG)
- net PG: now also IC2.4 (PG), R15.1, R18.1
- net at U14.5 (FB): now also R16.1, R17.2
- net at U14.6 (VCC): now also C15.1, R15.2
- net at U14.7 (BOOT): now also C16.2
- net at U14.8 (SW): now also C16.1, L1.1
- net at U11.22 (SCL): now also R37.1
- net at U11.23 (SDA): now also R36.1
- net at U11.3 (~{RESET}): now also R38.1
- net at IC2.5 (FB): now also R19.1, R20.2
- net at IC2.6 (VCC): now also C23.1, R18.2
- net at IC2.7 (BOOT): now also C24.2
- net at IC2.8 (SW): now also C24.1, L2.1
- net at U10.22 (SCL): now also R34.1
- net at U10.23 (SDA): now also R33.1
- net at U10.3 (~{RESET}): now also R35.1
- new net: C6.2, J6.2 (D-), R6.1
- new net: C5.2, J6.3 (D+), R4.1
- new net: C7.1, R4.1, R5.2, Y1.1
- new net: C4.1, R3.2, R4.2, Y1.2
- new net: C8.1, R7.1, SW1.2
- new net: R2.2, R45.1, R47.2
- new net: R46.1, R48.2, R49.1
- new net: C34.2, R46.2, U1.3 (VIN1P)
- new net: C19.2, C20.1
- new net: Q1.1, R24.2
- new net: C34.1, R45.2, U1.2 (VIN1N)
- new net: C27.2, C28.1
- new net: C17.2, C18.1
- new net: C18.2, C19.1
- new net: C35.1, U1.6 (VBG)
- new net: R39.1, U12.23 (SDA)
- new net: C25.2, C26.1
- new net: C26.2, C27.1
- new net: C32.1, C33.1, R2.1, R49.2, U1.1 (REFP), U1.16 (AVDD/LDO)
- new net: R40.1, U12.22 (SCL)
- new net: R41.1, U12.3 (~{RESET})
- new net -3V3: C25.1, L2.2, R19.2
- new net -5V: C17.1, L1.2, R16.2
- new net Boot: J7.1 (Pin_1), U8.27 (IO0)
- new net EN: C2.2, R1.1, R7.2, U8.3 (EN)
- new net IO15: R3.1, U8.8 (IO15)
- new net IO16: R5.1, U8.9 (IO16)
- new net RXD0: J16.3 (Pin_3), U8.36 (RXD0)
- new net TCK: J15.4 (Pin_4), U8.32 (IO39)
- new net TDI: J15.2 (Pin_2), U8.34 (IO41)
- new net TDO: J15.3 (Pin_3), U8.33 (IO40)
- new net TMS: J15.1 (Pin_1), U8.35 (IO42)
- new net TXD0: J16.2 (Pin_2), U8.37 (TXD0)
- new net USB_D+: R4.2, U8.14 (IO20)
- new net USB_D-: R6.2, U8.13 (IO19)
- no-connect marks 2 -> 15
Other:
- removed sheet Main_Floor_PCB
- note added: "Clamped at 36V"
- note added: "ESP32-S3-WROOM-1U Peripherals"
- note added: "TCA9548A Pull-up Out"
- note removed: "MCU+passives"
- moved on the sheet: IC1, J2, J5, U2, U3, U4

Commit message: Hardware Week 2
Parts:
- removed C14, C21: 10uF, symbol Device:C_Polarized
- removed C15, C23, C32, C33: 1uF, symbol Device:C_Polarized
- removed C17, C18, C19, C20, C25, C26, C27, C28: 22uF, symbol Device:C_Polarized
- removed J2, J5: Magnetic THT Pins Female, symbol Connector:DA15_Pins_MountingHoles
- removed R4 (x2): TBD, symbol Device:R
- removed U1: NAU7802SGI, NAU7802SGI:SOIC127P600X175-16N, symbol NAU7802SGI:NAU7802SGI
- removed U10: TCA9548APWR, TCA9548APWR:SOP65P640X120-24N, symbol TCA9548APWR:TCA9548APWR
- removed Z1: DDZ9702T-7, DDZ9702T7, symbol DDZ9702T-7:DDZ9702T-7
- added C14, C17: 10uF, symbol Device:C
- added C15, C21, C37: 1uF, symbol Device:C
- added C18, C19, C20, C32, C33, C38, C39, C40: 22uF, symbol Device:C
- added C23, C36: 100nF, symbol Device:C
- added C41: 47nF, symbol Device:C
- added D1: 1N4148W, Diode_SMD:D_SOD-123, symbol Diode:1N4148W
- added R4: TBD, symbol Device:R
- added R50: 43.3K, symbol Device:R
- added R51: 100, symbol Device:R
- added R52: 1K, symbol Device:R
- added R53: 1M, symbol Device:R
- added R54: 10K, symbol Device:R
- added R55: 100K, symbol Device:R
- added U10: NAU7802SGI, NAU7802SGI:SOIC127P600X175-16N, symbol NAU7802SGI:NAU7802SGI
- added U16: TCA9548APWR, TCA9548APWR:SOP65P640X120-24N, symbol TCA9548APWR:TCA9548APWR
- added Z3: DDZ9702T-7, DDZ9702T7, symbol DDZ9702T-7:DDZ9702T-7
- C29: value 100nF -> 47nF
- C30: value 100uF -> 220uF
- L2: value 8uH, 14mΩ -> 6.8uH, 14mΩ
- R14: value 10 -> TBD
- R15: value 100K -> 10
- R17: value 24.9K -> 100K
- R18: value 100K -> 24.9K
- R20: value 43.3K -> 100K
- R21: value 3.01K -> 10K
- R23: value 100K -> 243K
- R25: value 15m -> 6m
- R26: value 110K -> 115K
- R27: value 4.02K -> 4.99K
Connections:
- net +24V: now also C14.2, R52.2, R55.2; no longer U14.3 (EN), U15.8 (VCC)
- net +3V3: now also L2.2, R15.2, R20.2, C33.2, C38.2, C39.2, C40.2, R54.2, U10.15 (DVDD); no longer R14.2
- net +5V: now also L1.2, R17.2, C17.2, C18.2, C19.2, C20.2, C32.2, U16.24 (VCC)
- net EN: now also R14.2; no longer R7.2
- net GND: now also R18.1, C14.1, C15.2, C17.1, C18.1, C19.1, C20.1, C21.1, C23.2, C32.1, C33.1, C36.2, C37.2, C38.1, C39.1, C40.1, C41.2, R50.1, U10.7 (REFN), U10.8 (AVSS), U10.9 (DVSS), U16.1 (A0), U16.12 (GND), U16.2 (A1), U16.21 (A2); no longer R17.1, R20.1
- net PG: now also R16.1, R19.1; no longer R15.1, R18.1
- net TCA9548A SCX: now also U16.10 (SD3), U16.11 (SC3), U16.13 (SD4), U16.15 (SD5), U16.16 (SC5), U16.17 (SD6), U16.18 (SC6), U16.19 (SD7), U16.20 (SC7), U16.4 (SD0), U16.5 (SC0), U16.6 (SD1), U16.7 (SC1), U16.8 (SD2), U16.9 (SC2)
- net USB_D+: now also R6.2
- net USB_D-: now also R7.2; no longer R6.2
- net at C6.2, J6.2 (D-): now also R7.1; no longer R6.1
- net at C5.2, J6.3 (D+): now also R6.1
- net at U11.22 (SCL): now also R34.1; no longer R37.1
- net at R36.1: now also U12.23 (SDA); no longer U11.23 (SDA)
- net at R38.1: now also U12.3 (~{RESET}); no longer U11.3 (~{RESET})
- net at C7.1, R5.2, Y1.1: now also R4.1
- net at U14.6 (VCC): now also R16.2, C15.1; no longer R15.2
- net at C4.1, R3.2, Y1.2: now also R4.2
- net at C8.1, SW1.2: now also R14.1; no longer R7.1
- net at R33.1: now also U11.23 (SDA)
- net at R35.1: now also U11.3 (~{RESET})
- net at Q1.3, Q2.1 (S_1), U15.5 (SOURCE)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: now also Z3.2 (A)
- net at C34.2, R46.2: now also U10.3 (VIN1P)
- net at C11.1, C12.1, U4.2 (VDD): now also R15.1; no longer R14.1
- net at C34.1, R45.2: now also U10.2 (VIN1N)
- net at R18.2: now also R17.1, U14.5 (FB); no longer IC2.6 (VCC)
- net GPIO_X: now reaches U15.13 (*FLT)
- net GPIO_X: now also R54.1
- net EN_PS2: now reaches U15.14 (ENOUT)
- net EN_PS2: now also U14.3 (EN), R55.1
- net at R24.1, U15.6 (HGATE): now also D1.2 (A), R51.2, Z3.1 (K)
- net at U15.9 (*SHDN): now also R53.1
- net at C35.1: now also U10.6 (VBG)
- net at R39.1: now also U16.23 (SDA); no longer U12.23 (SDA)
- net at R2.1, R49.2: now also C36.1, C37.1, U10.1 (REFP), U10.16 (AVDD/LDO)
- net at R40.1: now also U16.22 (SCL); no longer U12.22 (SCL)
- net at R41.1: now also U16.3 (~{RESET}); no longer U12.3 (~{RESET})
- net SDA_0: now reaches U8.12 (IO8)
- net SDA_1: now reaches U8.15 (IO3)
- net SCL_0: now reaches U8.17 (IO9)
- net SCL_1: now reaches U8.4 (IO4)
- net -3V3: no longer names the net of R19.2
- net -3V3: now also IC2.6 (VCC), C21.2; no longer L2.2
- removed net -5V: L1.2, R16.2
- new net: C41.1, D1.1 (K), R51.1
- new net: C23.1, R52.1, R53.2, U15.8 (VCC)
- new net: IC2.5 (FB), R20.1, R50.2
- new net: R37.1, U12.22 (SCL)
- no-connect marks 15 -> 17
Other:
- note added: "Clamped at 32V"
- note added: "I2C Mux"
- note added: "Power Management 24V->5V 5V-3V3 Input Protection Controller Input current monitor"
- note removed: "Clamped at 36V"
- note removed: "Power Management 24V->5V 5V-3V3"

Commit message: schematic newest
Parts:
- removed C2, C5, C6: TBD, symbol Device:C
- removed C4, C7: 12pF, symbol Device:C
- removed J15: JTAG, symbol Connector:Conn_01x04_Pin
- removed J6: USB_OTG, symbol Connector:USB_OTG
- removed J7: Boot Option, symbol Connector:Conn_01x02_Pin
- removed R1, R3, R4, R5, R6, R7: TBD, symbol Device:R
- removed U11, U12, U16: TCA9548APWR, TCA9548APWR:SOP65P640X120-24N, symbol TCA9548APWR:TCA9548APWR
- removed Y1: 32.768KHz, symbol Device:Crystal
- added C42: 4.7uF, symbol Device:C
- added C43, C45, C52, C61, C62: 100nF, symbol Device:C
- added C44, C63: 1uF, symbol Device:C
- added C46, C47: 10nF, symbol Device:C
- added C48: 1nF, symbol Device:C
- added C49: 4.7nF, symbol Device:C
- added C50, C51: 220nF, symbol Device:C
- added C64: 470uF, symbol Device:C
- added D2: 40V 1A, symbol Device:D_Schottky
- added D4: SK6812, SK6812:LED_SK6812, symbol SK6812:SK6812
- added D7: ESD5Zxx, Diode_SMD:D_SOD-523, symbol Diode:ESD5Zxx
- added D8: SMBJ33A, SMBJ33A-13-F:DIOM5336X250N, symbol SMBJ33A-13-F:SMBJ33A-13-F
- added J15: Molex Micro-Fit 3.0, 0430451213, symbol 0430451213:0430451213
- added J2: KPJX-4S, KPJX-4S:KYCON_KPJX-4S, symbol KPJX-4S:KPJX-4S
- added J5: 2495155-1, 2495155-1:TE_2495155-1, symbol 2495155-1:2495155-1
- added R56: 4.87K, symbol Device:R
- added R57: 1.2K, symbol Device:R
- added R58: 802, symbol Device:R
- added R59, R60: 4.7K, symbol Device:R
- added R61: 100K, symbol Device:R
- added SW2: SW_Push, symbol Switch:SW_Push
- added SW3: SW_Reed, symbol Switch:SW_Reed
- added U11: TPS27S100BPWPR, TPS27S100BPWPR:IC_TPS27S100BPWPR, symbol TPS27S100BPWPR:TPS27S100BPWPR
- added U24: USBLC6-2P6, USBLC6-2P6:SOT50P160X60-6N, symbol USBLC6-2P6:USBLC6-2P6
- added U26, U27, U28: P82B96D, P82B96D:SOIC127P599X175-8N, symbol P82B96D:P82B96D
- C8: value TBD -> 1uF
- L1: value 8uH, 14mΩ -> 8.2uH, 14mΩ
- R12, R13: value 2.2K -> 4.7K
- R14: value TBD -> 10K
- R19: value 100K -> 5.1K
- R28, R29, R31, R32, R33, R34, R42, R43: value 10K -> 4.7K
- R35: value 10K -> 100K
- R36: value 10K -> 5.1K
- R40: value 10K -> 47
- R45, R46: value 47 -> 100
Connections:
- net IO15 is gone; now on net LOADCELL_DRDY: U8.8 (IO15)
- net IO16 is gone; now on net SDA_1: U8.9 (IO16)
- net TCK is gone; now on net VIN_FLT_N: U8.32 (IO39)
- net TDO is gone; now on net PG_5V: U8.33 (IO40)
- net +24V: now also C42.2, C49.2, C50.2, C51.2, C62.1, D2.1 (K), D8.1, J2.1, J2.4, U11.10 (IN), U11.5 (OUT), U11.6 (OUT), U11.7 (OUT), U11.8 (IN), U11.9 (IN)
- net +3V3: now also C31.1, R14.2, R16.2, R31.1, R32.1, R33.1, R34.1, R37.1, R38.1, R42.1, R43.1, R44.1, U13.6 (VS), U9.1 (A0), U9.2 (A1), U9.21 (A2), U9.24 (VCC), C43.2, C44.1, C45.1, R59.1; no longer R33.2, R34.2, R35.2, R36.2, R37.2, R38.2, R39.2, R40.2
- net +5V: now also IC1.14 (VCC), R35.1, C52.2, C61.1, C63.2, C64.2, D2.2 (A), D4.1 (VDD), U28.8 (VCC); no longer C31.1, IC2.3 (EN), R31.1, R32.1, R42.1, R43.1, R44.1, U13.6 (VS), U9.24 (VCC)
- net Boot: now also R41.1, SW2.2
- net EN: now also C8.1, IC2.4 (PG), R14.1, SW1.2; no longer R14.2
- net SCL: no longer R12.2, U4.1 (SCL)
- net SCL_0: now also R29.1, U8.25 (IO48), U9.22 (SCL); no longer U8.17 (IO9)
- net SCL_1: now also R12.2, R34.2, R43.2, U10.13 (SCLK), U13.5 (SCL), U4.1 (SCL), U8.10 (IO17); no longer U8.4 (IO4)
- net SDA: no longer R13.2, U4.4 (SDA)
- net SDA_0: now also R28.1, U8.24 (IO47), U9.23 (SDA); no longer U8.12 (IO8)
- net SDA_1: now also R13.2, R33.2, R42.2, U10.14 (SDIO), U13.4 (SDA), U4.4 (SDA); no longer U8.15 (IO3)
- net USB_D+: now also U24.4
- net USB_D-: now also U24.6
- net at C21.2, IC2.6 (VCC): no longer R19.2
- net at C34.2, R46.2, U10.3 (VIN1P): now also C47.1
- net at C34.1, R45.2, U10.2 (VIN1N): now also C46.1
- net at R36.1: now also J5.A5 (CC1)
- net at R40.1: now also IC1.3 (1Y)
- net EXP: now reaches R39.1
- net EXP: now also C1.2, C10.1, C11.2, C12.2, C13.1, C14.1, C15.2, C17.1, C18.1, C19.1, C20.1, C21.1, C22.1, C23.2, C29.2, C3.2, C30.2, C31.2, C32.1, C33.1, C35.2, C36.2, C37.2, C38.1, C39.1, C40.1, C41.2, C8.2, C9.2, IC1.1 (1~{OE}), IC1.10 (3~{OE}), IC1.12 (4A), IC1.13 (4~{OE}), IC1.4 (2~{OE}), IC1.5 (2A), IC1.7 (GND), IC1.9 (3A), IC2.1 (PGND), IC2.9 (EP), J16.4 (Pin_4), R18.1, R19.2, R21.1, R27.1, R36.2, R47.1, R48.1, R50.1, SW1.1, U10.10 (XIN), U10.7 (REFN), U10.8 (AVSS), U10.9 (DVSS), U13.1 (A1), U13.2 (A0), U13.7 (GND), U14.1 (PGND), U14.9 (AGND), U15.12 (GND), U2.20 (GND), U2.21 (GND), U2.6 (GND), U3.4 (VSS), U4.3 (GND), U8.1 (GND), U8.40 (GND), U8.41_1 (GND), U8.41_2 (GND), U8.41_3 (GND), U8.41_4 (GND), U8.41_5 (GND), U8.41_6 (GND), U8.41_7 (GND), U8.41_8 (GND), U8.41_9 (GND), U9.12 (GND), C42.1, C43.1, C44.2, C45.2, C46.2, C47.2, C48.1, C49.1, C50.1, C51.1, C52.1, C61.2, C62.2, C63.1, C64.1, D4.3 (VSS), D7.2 (A), D8.2, J2.S1 (SHIELD), J5.A1/B12 (GND_A), J5.B1/A12 (GND_B), J5.SH1 (SHIELD), J5.SH2 (SHIELD), J5.SH3 (SHIELD), J5.SH4 (SHIELD), R56.1, R57.2, R61.2, SW2.1, U11.15 (EXP), U11.16 (EXP), U11.17 (EXP), U11.18 (EXP), U11.19 (EXP), U11.2 (GND), U11.20 (EXP), U11.21 (EXP)
- net PG_5V: now reaches C15.1, U14.6 (VCC)
- net PG_5V: now also R16.1, U14.4 (PG); no longer R16.2
- net PWR_ALERT_N: now reaches U8.11 (IO18)
- net PWR_ALERT_N: now also R44.2, U13.3 (ALERT)
- net nRESET_DRV: now reaches U8.16 (IO46)
- net OW_F1: now reaches U8.19 (IO11)
- net OW_F2: now reaches U8.20 (IO12)
- net OW_F3: now reaches U8.21 (IO13)
- net LEAK_EXC: now reaches U8.22 (IO14)
- net MUX_RST_N: now reaches U8.23 (IO21)
- net MUX_RST_N: now also R30.1, U9.3 (~{RESET})
- net OE_DRV: now reaches U8.26 (IO45)
- net VALVE_RAIL_EN: now reaches U8.31 (IO38)
- net VALVE_RAIL_EN: now also R60.1
- net VALVE_IMON: now reaches U8.5 (IO5)
- net VALVE_IMON: now also C48.2, R58.1
- net VALVE_RAIL_SENSE: now reaches U8.6 (IO6)
- net LEAK_BASE: now reaches U8.7 (IO7)
- net RING_DATA: now reaches IC1.2 (1A)
- net RING_DATA: now also R39.2, U8.12 (IO8)
- net TCA9548A SCX >2: now reaches U9.14 (SC4)
- net TCA9548A SCX >2: now also R38.2, U9.11 (SC3), U9.16 (SC5), U9.18 (SC6), U9.20 (SC7), U9.9 (SC2)
- net LOADCELL_DRDY: now reaches U10.12 (DRDY)
- removed net GND: C1.2, C10.1, C11.2, C12.2, C13.1, C14.1, C15.2, C17.1, C18.1, C19.1, C20.1, C21.1, C22.1, C23.2, C29.2, C3.2, C30.2, C31.2, C32.1, C33.1, C35.2, C36.2, C37.2, C38.1, C39.1, C40.1, C41.2, C8.2, C9.2, IC2.1 (PGND), IC2.9 (EP), J16.4 (Pin_4), R18.1, R21.1, R27.1, R47.1, R48.1, R50.1, SW1.1, U10.7 (REFN), U10.8 (AVSS), U10.9 (DVSS), U13.7 (GND), U14.1 (PGND), U14.9 (AGND), U15.12 (GND), U2.20 (GND), U2.21 (GND), U2.6 (GND), U3.4 (VSS), U4.3 (GND), U8.1 (GND), U8.40 (GND), U8.41_1 (GND), U8.41_2 (GND), U8.41_3 (GND), U8.41_4 (GND), U8.41_5 (GND), U8.41_6 (GND), U8.41_7 (GND), U8.41_8 (GND), U8.41_9 (GND), U9.1 (A0), U9.12 (GND), U9.2 (A1), U9.21 (A2)
- net GPIO_X renamed VIN_FLT_N
- removed net PG: IC2.4 (PG), R16.1, R19.1, U14.4 (PG)
- removed net TCA9548A SCX: R31.2, R32.2, U9.10 (SD3), U9.11 (SC3), U9.13 (SD4), U9.15 (SD5), U9.16 (SC5), U9.17 (SD6), U9.18 (SC6), U9.19 (SD7), U9.20 (SC7), U9.4 (SD0), U9.5 (SC0), U9.6 (SD1), U9.7 (SC1), U9.8 (SD2), U9.9 (SC2)
- net TDI renamed PUMP_EN
- net TMS renamed TANK_LOW
- new net: R60.2, R61.1, U11.3 (EN)
- new net: R56.2, U11.13 (ILIM)
- new net: R59.2, U11.12 (DIAG_EN)
- new net: R57.1, R58.2, U11.14 (IMON)
- new net: J5.B5 (CC2), R19.1
- new net: IC2.3 (EN), R35.2
- new net: J5.A7 (DN1), U24.1
- new net: J5.A6 (DP1), U24.3
- new net 1Y_out: D4.4 (DIN), D7.1 (K), R40.2
- new net Earth_Protective: J2.2, J2.3
- new net TCA9548A SCX <3: R32.2, U9.5 (SC0), U9.7 (SC1)
- new net TCA9548A SDX <3: R31.2, U9.4 (SD0), U9.6 (SD1)
- new net TCA9548A SDX >2: R37.2, U9.10 (SD3), U9.13 (SD4), U9.15 (SD5), U9.17 (SD6), U9.19 (SD7), U9.8 (SD2)
- new net V24_SENSE: U8.4 (IO4)
- no-connect marks 17 -> 29
Other:
- note added: "Floor cabling needs revision"
- note added: "INA226AIDGSR comes after LTC4364IS"
- note added: "In reality 2 "Basic Floor" will be printed"
- note added: "TCA9548A Pull-up Out 0-2"
- note added: "TCA9548A Pull-up Out 3-7"
- note removed: "TCA9548A Pull-up Out"
