File: Hardware/Main_PCB/GrowHub_Elec.kicad_sch (KiCad schematic)
At the start: 136 parts, among them IC1 74AHCT125D,118, IC2 LMR33610BDDAR, J15 Molex Micro-Fit 3.0, J16 JTAG, J2 KPJX-4S, J5 2495155-1, Q1 FDB3632, Q2 FDMS86101, SW1 SW_Push, SW2 SW_Push, SW3 SW_Reed, U10 NAU7802SGI, U11 TPS27S100BPWPR, U13 INA226AIDGSR, U14 LMR33630ADDA, U15 LTC4364IS-2_PBF, U2 SCD41-D-R2, U24 USBLC6-2P6, U26 P82B96D, U27 P82B96D, U28 P82B96D, U3 SHT4XI-DIGITAL, U4 VEML7700-TT, U8 ESP32-S3-WROOM-1U-N16R8, U9 TCA9548APWR

Commit message: Week 4 Schematic
Parts:
- removed C10, C3: 100nF, symbol Device:C
- removed C64: 470uF, symbol Device:C
- removed C9: 22uF, symbol Device:C_Polarized
- removed IC2: LMR33610BDDAR, LMR33610BDDAR:LMR33610BDDAR, symbol LMR33610BDDAR:LMR33610BDDAR
- removed J16: JTAG, symbol Connector:Conn_01x04_Pin
- removed R10, R11, R14, R8, R9: 10K, symbol Device:R
- removed U2: SCD41-D-R2, SCD41-D-R2:XDCR_SCD41-D-R2, symbol SCD41-D-R2:SCD41-D-R2
- removed U26, U27, U28: P82B96D, P82B96D:SOIC127P599X175-8N, symbol P82B96D:P82B96D
- removed U3: SHT4XI-DIGITAL, SHT4XI-DIGITAL:SHT4XI-DIGITAL, symbol SHT4XI-DIGITAL:SHT4XI-DIGITAL
- added C2: 22uF, symbol Device:C_Polarized
- added C4, C5, C6: 10nF, symbol Device:C
- added C67, C7, C71, C82, C83: 100nF, symbol Device:C
- added C72: 330pF, symbol Device:C
- added C9: 47nF, symbol Device:C
- added D10, D11, D12, D13, D14, D15, D16, D17, D18, D25, D26, D3, D32, D33, D37, D38, D39, D5: ESD5Zxx, Diode_SMD:D_SOD-523, symbol Diode:ESD5Zxx
- added F1: Polyfuse, symbol Device:Polyfuse
- added J17, J18: Molex Micro-Fit 3.0, 0430451213, symbol 0430451213:0430451213
- added PS3: LMR33610ADDAR, SOIC127P600X170-9N, symbol LMR33610ADDAR:LMR33610ADDAR
- added Q10, Q11, Q12, Q13, Q14, Q20, Q21, Q8, Q9: BSS138BK-215, TL431CDBZR215, symbol BSS138BK-215:BSS138BK-215
- added R100, R85, R86, R87, R98: 1K, symbol Device:R
- added R119, R120, R121, R122, R123, R124, R97: 0, symbol Device:R
- added R129, R130, R133, R134, R137, R138, R77, R89, R90, R91, R92, R93, R99: 10K, symbol Device:R
- added R131, R132, R135, R136, R139, R140: R_pu, symbol Device:R
- added R66, R72, R75, R76, R78, R79, R81, R83: 100K, symbol Device:R
- added R80: 4.7K, symbol Device:R
- added R82: 5.6K, symbol Device:R
- added R84: 8.2K, symbol Device:R
- added R95, R96: 10, symbol Device:R
- added SW4: SW_DIP_x01, symbol Switch:SW_DIP_x01
- added U1, U2, U5: PCA9600DPZ, TSSOP8_PCA9600_NXP, symbol 2026-10-11_13-08-00:PCA9600DPZ
- C1: value 22uF -> 470uF
- C63: value 1uF -> 100nF
- R25: value 6m -> 5m
- R42: value 4.7K -> 10K
- R43: value 4.7K -> 0
- R50: value 43.3K -> 43.2K
- R58: value 802 -> 820
Connections:
- net +24V: now also R96.2; no longer C51.2, U11.5 (OUT), U11.6 (OUT), U11.7 (OUT)
- net +3V3: now also Q13.1 (G), Q14.1 (G), Q21.1 (G), R129.1, R130.1, R133.1, R134.1, R137.1, R138.1, R77.1, R80.2, R89.1, R90.1, R91.1, R92.1, R93.1; no longer C1.1, R42.1, R43.1, U8.2 (3V3)
- net +5V: now also C52.1, C61.2, J15.10 (10_5V), J15.9 (9_5V), C82.2, C83.2, F1.1, J17.10 (10_5V), J17.9 (9_5V), J18.10 (10_5V), J18.9 (9_5V), PS3.2 (VIN), R131.1, R132.1, R135.1, R136.1, R139.1, R140.1, U1.8 (VCC), U2.8 (VCC), U5.8 (VCC); no longer C52.2, C61.1, C63.2, D4.1 (VDD)
- net Boot: now also C9.1
- net EN: now also R42.2, PS3.4 (PG)
- net EXP: now also C52.2, C61.1, J15.7 (7_GND), J15.8 (8_GND), C2.2, C4.2, C5.2, C6.2, C67.2, C7.2, C82.1, C83.1, C9.2, D10.2 (A), D11.2 (A), D12.2 (A), D13.2 (A), D14.2 (A), D15.2 (A), D16.2 (A), D17.2 (A), D18.2 (A), D25.2 (A), D26.2 (A), D3.2 (A), D32.2 (A), D33.2 (A), D37.2 (A), D38.2 (A), D39.2 (A), D5.2 (A), J17.7 (7_GND), J17.8 (8_GND), J18.7 (7_GND), J18.8 (8_GND), PS3.1 (PGND), PS3.9 (EP), Q10.2 (S), Q11.2 (S), Q12.2 (S), Q20.2 (S), Q8.2 (S), Q9.2 (S), R66.2, R72.2, R75.2, R76.2, R78.2, R79.2, R82.1, R84.2, R99.1, SW4.1, U1.4 (GND), U2.4 (GND), U5.4 (GND); no longer C52.1, C61.2
- net OE_DRV: now also Q10.1 (G), Q20.1 (G), Q8.1 (G), R75.1, R76.1, R79.1
- net OW_F1: now also Q13.2 (S), R77.2
- net OW_F2: now also Q21.2 (S), R90.2
- net OW_F3: now also Q14.2 (S), R92.2
- net PG_5V: no longer C15.1, U14.6 (VCC)
- net SCL_1: no longer R43.2
- net SDA_1: no longer R42.2
- net TANK_LOW: now also C67.1, R100.2
- net TCA9548A SCX <3: no longer U9.5 (SC0), U9.7 (SC1)
- net TCA9548A SCX >2: no longer U9.9 (SC2)
- net TCA9548A SDX <3: no longer U9.4 (SD0), U9.6 (SD1)
- net TCA9548A SDX >2: no longer U9.8 (SD2)
- net USB_D+: now also R43.1; no longer U24.4
- net USB_D-: now also R97.1; no longer U24.6
- net V24_SENSE: now also C4.1, R81.2, R85.1
- net VALVE_IMON: now also C6.1, R87.1, R87.2, R98.1; no longer R58.1
- net nRESET_DRV: now also Q11.1 (G), Q12.1 (G), Q9.1 (G), R66.1, R72.1, R78.1
- net at R2.2, R45.1, R47.2: now also D25.1 (K)
- net at R58.2, U11.14 (IMON): no longer R57.1
- net IN+: now reaches Q2.5 (D_1), R25.2, U15.2 (SENSE)
- net IN+: now also R95.2
- net HGATE: now reaches D1.2 (A), R24.1, U15.6 (HGATE), Z3.1 (K)
- net HGATE: now also R51.1; no longer R51.2
- net at C41.1, D1.1 (K): now also R51.2; no longer R51.1
- net at R20.1, R50.2: now also PS3.5 (FB)
- net at SW3.1: now also SW4.2
- net at SW3.2: now also D3.1 (K), R100.1, R80.1
- net at U10.4 (VIN2N): now also C72.1
- net at U10.5 (VIN2P): now also C72.2
- net at R46.1, R48.2, R49.1: now also D26.1 (K)
- net at C24.1, L2.1: now also PS3.8 (SW)
- net at C21.2: now also PS3.6 (VCC)
- net at C24.2: now also PS3.7 (BOOT)
- net at R35.2: now also PS3.3 (EN)
- net at U13.10 (IN+): now also C71.1, R95.1
- net at U13.9 (IN-): now also C71.2, R96.1
- net OE_1: now reaches J15.1
- net OE_1: now also D10.1 (K), Q8.3 (D)
- net 1-Wire_1: now reaches J15.11
- net 1-Wire_1: now also D12.1 (K), Q13.3 (D), R89.2
- net nRESET_1: now reaches J15.2
- net nRESET_1: now also D11.1 (K), Q11.3 (D), Q12.3 (D), Q9.3 (D)
- net SCL_F1: now reaches J15.3
- net SCL_F1: now also D5.1 (K), R120.2, R132.2, U1.5 (TY), U1.6 (RY)
- net SDA_F1: now reaches J15.4
- net SDA_F1: now also D37.1 (K), R119.1, R131.2, U1.2 (RX), U1.3 (TX)
- net VALVE_RAIL: now reaches J15.5
- net VALVE_RAIL: now also C51.2, U11.5 (OUT), U11.6 (OUT), U11.7 (OUT), J17.5, J18.5, R83.1, R99.2
- net VALVE_RAIL_SENSE renamed VALVE_RAIL_SENSE_DIV
- net VALVE_RAIL_SENSE_DIV: now also C5.1, R86.2
- new net: C1.1, C63.2, D4.1 (VDD), F1.2
- new net: R97.2, U24.6
- new net: R43.2, U24.4
- new net: C15.1, U14.6 (VCC)
- new net: R57.1, R58.1, R98.2
- new net: R83.2, R84.1, R86.1
- new net: R81.1, R82.2, R85.2
- new net 1-Wire_2: D15.1 (K), J17.11, Q21.3 (D), R91.2
- new net 1-Wire_3: D18.1 (K), J18.11, Q14.3 (D), R93.2
- new net 3V3: C2.1, C7.1, R42.1, U8.2 (3V3)
- new net OE_2: D14.1 (K), J17.1, Q10.3 (D)
- new net OE_3: D17.1 (K), J18.1, Q20.3 (D)
- new net SCL_F2: D32.1 (K), J17.3, R122.2, R135.2, U2.5 (TY), U2.6 (RY)
- new net SCL_F3: D33.1 (K), J18.3, R124.2, R139.2, U5.5 (TY), U5.6 (RY)
- new net SC_0: R120.1, R129.2, U1.7 (SY), U9.5 (SC0)
- new net SC_1: R122.1, R133.2, U2.7 (SY), U9.7 (SC1)
- new net SC_2: R124.1, R137.2, U5.7 (SY), U9.9 (SC2)
- new net SDA_F2: D38.1 (K), J17.4, R121.1, R136.2, U2.2 (RX), U2.3 (TX)
- new net SDA_F3: D39.1 (K), J18.4, R123.1, R140.2, U5.2 (RX), U5.3 (TX)
- new net SD_0: R119.2, R130.2, U1.1 (SX), U9.4 (SD0)
- new net SD_1: R121.2, R134.2, U2.1 (SX), U9.6 (SD1)
- new net SD_2: R123.2, R138.2, U5.1 (SX), U9.8 (SD2)
- new net nRESET_2: D13.1 (K), J17.2
- new net nRESET_3: D16.1 (K), J18.2
- no-connect marks 29 -> 27
Other:
- note added: "100V X7R"
- note added: "Driver FETs"
- note added: "E+"
- note added: "E-"
- note added: "In reality 3 "Basic Floor" will be printed"
- note added: "Load Cell"
- note added: "Magnet float switch Closed when wet"
- note added: "Out of PCB"
- note added: "Pull-ups might be present at diff location"
- note added: "S+"
- note added: "S-"
- note added: "Use separate via GND for each"
- note removed: "In reality 2 "Basic Floor" will be printed"
- moved on the sheet: C11, C12, C13, C14, C15, C16, C17, C18, C19, C20, C21, C22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

Commit message: Finished schematics
Parts:
- removed C1: 470uF, symbol Device:C_Polarized
- removed C11: 10uF, symbol Device:C_Polarized
- removed C2: 22uF, symbol Device:C_Polarized
- removed C21: 1uF, symbol Device:C
- removed C30: 220uF, symbol Device:C_Polarized
- removed C36, C61, C62, C63, C67, C71: 100nF, symbol Device:C
- removed C72: 330pF, symbol Device:C
- removed D1: 1N4148W, Diode_SMD:D_SOD-123, symbol Diode:1N4148W
- removed D10, D11, D12, D15, D16, D25, D26, D3, D32, D33, D37, D38, D5: ESD5Zxx, Diode_SMD:D_SOD-523, symbol Diode:ESD5Zxx
- removed D2: 40V 1A, symbol Device:D_Schottky
- removed D4: SK6812, SK6812:LED_SK6812, symbol SK6812:SK6812
- removed D8: SMBJ33A, SMBJ33A-13-F:DIOM5336X250N, symbol SMBJ33A-13-F:SMBJ33A-13-F
- removed F1: Polyfuse, symbol Device:Polyfuse
- removed IC1: 74AHCT125D,118, SOIC127P600X175-14N, symbol 74AHCT125D_118:74AHCT125D,118
- removed J15, J17, J18: Molex Micro-Fit 3.0, 0430451213, symbol 0430451213:0430451213
- removed J2: KPJX-4S, KPJX-4S:KYCON_KPJX-4S, symbol KPJX-4S:KPJX-4S
- removed J5: 2495155-1, 2495155-1:TE_2495155-1, symbol 2495155-1:2495155-1
- removed PS3: LMR33610ADDAR, SOIC127P600X170-9N, symbol LMR33610ADDAR:LMR33610ADDAR
- removed Q1: FDB3632, FDB3632:TO254P1524X483-3N, symbol FDB3632:FDB3632
- removed Q10, Q11, Q12, Q13, Q14, Q20, Q21, Q8, Q9: BSS138BK-215, TL431CDBZR215, symbol BSS138BK-215:BSS138BK-215
- removed Q2: FDMS86101, FDMS86252, symbol FDMS86101:FDMS86101
- removed R100, R86, R87, R98: 1K, symbol Device:R
- removed R129, R130, R133, R134, R137, R138, R99: 10K, symbol Device:R
- removed R131, R132, R135, R136, R139, R140: R_pu, symbol Device:R
- removed R24, R95, R96: 10, symbol Device:R
- removed R25: 5m, symbol Device:R
- removed R47, R48, R49: R_45deg, symbol Device:R_45deg
- removed R97: 0, symbol Device:R
- removed SW3: SW_Reed, symbol Switch:SW_Reed
- removed SW4: SW_DIP_x01, symbol Switch:SW_DIP_x01
- removed U1, U2, U5: PCA9600DPZ, TSSOP8_PCA9600_NXP, symbol 2026-10-11_13-08-00:PCA9600DPZ
- removed U10: NAU7802SGI, NAU7802SGI:SOIC127P600X175-16N, symbol NAU7802SGI:NAU7802SGI
- removed U11: TPS27S100BPWPR, TPS27S100BPWPR:IC_TPS27S100BPWPR, symbol TPS27S100BPWPR:TPS27S100BPWPR
- removed U13: INA226AIDGSR, INA226AIDGSR:SOP50P490X110-10N, symbol INA226AIDGSR:INA226AIDGSR
- removed U14: LMR33630ADDA, LMR33630ADDA:VREG_LM5017MR_NOPB, symbol LMR33630ADDA:LMR33630ADDA
- removed U15: LTC4364IS-2_PBF, LTC4364IS-2_PBF:SO-16_S, symbol LTC4364IS-2_PBF:LTC4364IS-2_PBF
- removed U24: USBLC6-2P6, USBLC6-2P6:SOT50P160X60-6N, symbol USBLC6-2P6:USBLC6-2P6
- removed U4: VEML7700-TT, VEML7700-TT:XDCR_VEML7700-TT, symbol VEML7700-TT:VEML7700-TT
- removed U8: ESP32-S3-WROOM-1U-N16R8, ESP32-S3-WROOM-1U-N16R8:XCVR_ESP32-S3-WROOM-1U-N16R8, symbol ESP32-S3-WROOM-1U-N16R8:ESP32-S3-WROOM-1U-N16R8
- removed U9: TCA9548APWR, TCA9548APWR:SOP65P640X120-24N, symbol TCA9548APWR:TCA9548APWR
- removed Z2, Z3: DDZ9702T-7, DDZ9702T7, symbol DDZ9702T-7:DDZ9702T-7
- added C1, C10, C26, C27, C28, C79, C80, C81, C84: 100nF, Capacitor_SMD:C_0603_1608Metric, symbol Device:C
- added C11: 330pF, Capacitor_SMD:C_0603_1608Metric, symbol Device:C
- added C2: 1uF, Capacitor_SMD:C_0603_1608Metric, symbol Device:C
- added C25: 22nF, Capacitor_SMD:C_0603_1608Metric, symbol Device:C
- added C3, C53, C54: 22uF, Capacitor_SMD:C_1206_3216Metric, symbol Device:C
- added C30: 100nF, Capacitor_SMD:C_0805_2012Metric, symbol Device:C
- added C36: 220uF, Capacitor_SMD:CP_Elec_10x10.5, symbol Device:C_Polarized
- added D1, D2, D40, D42, D43: ESD5Z3.3T1G, Diode_SMD:D_SOD-523, symbol Diode:ESD5Zxx
- added D16: SS16, Diode_SMD:D_SMA, symbol Device:D_Schottky
- added D19, D20, D22, D41, D44, D8, D9: ESD5Z6.0T1G, Diode_SMD:D_SOD-523, symbol Diode:ESD5Zxx
- added D21: 1N4148W, Diode_SMD:D_SOD-123, symbol Diode:1N4148W
- added D23: SMBJ33A, Diode_SMD:D_SMB, symbol GrowHub:SMBJ33A-13-F
- added D34, D35, D36: SS16, Diode_SMD:D_SMA, symbol Diode:SS16
- added D37, D38, D4: SK6812, GrowHub:LED_SK6812, symbol GrowHub:SK6812
- added IC1: 74AHCT125D,118, Package_SO:SOIC-14_3.9x8.7mm_P1.27mm, symbol GrowHub:74AHCT125D,118
- added J1: USB-C 2495155-1, GrowHub:TE_2495155-1, symbol GrowHub:2495155-1
- added J10, J8, J9: VALVE(G88MPB02002C1EU), GrowHub:AMPHENOL_G88MPB02002C1EU, symbol GrowHub:G88MPB02002C1EU
- added J11: Load cell (JST PH 5p), Connector_JST:JST_PH_B5B-PH-K_1x05_P2.00mm_Vertical, symbol GrowHub:LoadCell_PH5
- added J13: Float S11 (JST PH 2p), Connector_JST:JST_PH_B2B-PH-K_1x02_P2.00mm_Vertical, symbol Connector:Conn_01x02_Pin
- added J14, J15, J4: Micro-Fit 3.0 2x6 (43045-1213), GrowHub:0430451213, symbol GrowHub:MicroFit3_2x06_FloorBus
- added J5: KPJX-4S (PSU DIN), GrowHub:KYCON_KPJX-4S, symbol GrowHub:KPJX-4S
- added PS1: LMR33610ADDAR, Package_SO:Texas_HSOP-8-1EP_3.9x4.9mm_P1.27mm_ThermalVias, symbol GrowHub:LMR33610ADDAR
- added Q1, Q2, Q3, Q4, Q5, Q6, Q7, Q8, Q9: BSS138BK-215, Package_TO_SOT_SMD:SOT-23, symbol GrowHub:BSS138BK-215
- added Q10: FDB3632, GrowHub:TO254P1524X483-3N, symbol GrowHub:FDB3632
- added Q11: FDMS86101, GrowHub:FDMS86252, symbol GrowHub:FDMS86101
- added Q18, Q19, Q20: AO3422, Package_TO_SOT_SMD:SOT-23, symbol GrowHub:AO3422
- added R1, R7, R8: LoadCell arm, symbol Device:R_45deg
- added R10, R11: 100K, Resistor_SMD:R_0603_1608Metric, symbol Device:R
- added R14: 100, Resistor_SMD:R_0603_1608Metric, symbol Device:R
- added R3, R48, R88: 10K, Resistor_SMD:R_0603_1608Metric, symbol Device:R
- added R4, R9: 4.7K, Resistor_SMD:R_0603_1608Metric, symbol Device:R
- added R47, R68, R69: 22K, Resistor_SMD:R_0603_1608Metric, symbol Device:R
- added R49, R5, R6, R71: 0, Resistor_SMD:R_0603_1608Metric, symbol Device:R
- added R62: 1M, Resistor_SMD:R_0603_1608Metric, symbol Device:R
- added R63: 1K, Resistor_SMD:R_0603_1608Metric, symbol Device:R
- added R64, R65: 2.2K, Resistor_SMD:R_0603_1608Metric, symbol Device:R
- added R67: 10, Resistor_SMD:R_0603_1608Metric, symbol Device:R
- added R70: 5m 1% 1W, Resistor_SMD:R_Shunt_Vishay_WSK2512_6332Metric_T1.19mm, symbol GrowHub:R_Shunt_Kelvin
- added R73: 115K, Resistor_SMD:R_0603_1608Metric, symbol Device:R
- added R74: 4.99K, Resistor_SMD:R_0603_1608Metric, symbol Device:R
- added R94: 43.2K, Resistor_SMD:R_0603_1608Metric, symbol Device:R
- added TP1: IO-0, TestPoint:TestPoint_Pad_D1.5mm, symbol Connector:TestPoint
- added U1: USBLC6-2P6, Package_TO_SOT_SMD:SOT-666, symbol GrowHub:USBLC6-2P6
- added U10: LMR33630ADDA, Package_SO:Texas_HSOP-8-1EP_3.9x4.9mm_P1.27mm_ThermalVias, symbol GrowHub:LMR33630ADDA
- added U11: INA226AIDGSR, Package_SO:VSSOP-10_3x3mm_P0.5mm, symbol GrowHub:INA226AIDGSR
- added U12: TCA9548APWR, Package_SO:TSSOP-24_4.4x7.8mm_P0.65mm, symbol GrowHub:TCA9548APWR
- added U2: VEML7700-TT, GrowHub:XDCR_VEML7700-TT, symbol GrowHub:VEML7700-TT
- added U3: NAU7802SGI, Package_SO:SOIC-16_3.9x9.9mm_P1.27mm, symbol GrowHub:NAU7802SGI
- added U4: TPS27S100BPWPR, GrowHub:IC_TPS27S100BPWPR, symbol GrowHub:TPS27S100BPWPR
- added U5, U7, U9: PCA9600DPZ, Package_SO:TSSOP-8_3x3mm_P0.65mm, symbol GrowHub:PCA9600DPZ
- added U6: ESP32-S3-WROOM-1U-N16R8, GrowHub:XCVR_ESP32-S3-WROOM-1U-N16R8, symbol GrowHub:ESP32-S3-WROOM-1U-N16R8
- added U8: LTC4364IS-2_PBF, Package_SO:SOIC-16_3.9x9.9mm_P1.27mm, symbol GrowHub:LTC4364IS-2_PBF
- added Z1, Z2: DDZ9702T-7, Diode_SMD:D_SOD-523, symbol GrowHub:DDZ9702T-7
- C12, C35, C7, C83: footprint (none) -> Capacitor_SMD:C_0603_1608Metric; Rating (none) -> 16V X7R
- C13: value 220nF -> 47nF; footprint (none) -> Capacitor_SMD:C_0603_1608Metric; Rating (none) -> 16V X7R
- C14: value 10uF -> 1uF; footprint (none) -> Capacitor_SMD:C_0603_1608Metric; Rating (none) -> 16V X7R
- C15, C37: value 1uF -> 100nF; footprint (none) -> Capacitor_SMD:C_0603_1608Metric; Rating (none) -> 16V X7R
- C16: value 100nF -> 10nF; footprint (none) -> Capacitor_SMD:C_0603_1608Metric; Rating (none) -> 16V X7R
- C17: value 10uF -> 100nF; footprint (none) -> Capacitor_SMD:C_0603_1608Metric; Rating (none) -> 16V X7R
- C18, C20: value 22uF -> 10nF; footprint (none) -> Capacitor_SMD:C_0603_1608Metric; Rating (none) -> 16V X7R
- C19: value 22uF -> 1nF; footprint (none) -> Capacitor_SMD:C_0603_1608Metric; Rating (none) -> 50V C0G
- C22, C50: value 220nF -> 100nF; footprint (none) -> Capacitor_SMD:C_0603_1608Metric; Rating (none) -> 16V X7R
- C23: value 100nF -> 220nF; footprint (none) -> Capacitor_SMD:C_0603_1608Metric; Rating (none) -> 50V X7R
- C24: value 100nF -> 4.7nF; footprint (none) -> Capacitor_SMD:C_0603_1608Metric; Rating (none) -> 50V X7R
- C29: value 47nF -> 10uF; footprint (none) -> Capacitor_SMD:C_1210_3225Metric; Rating (none) -> 50V X7R
- C31: value 100nF -> 4.7uF; footprint (none) -> Capacitor_SMD:C_1210_3225Metric; Rating (none) -> 50V X7R
- C32: value 22uF -> 220nF; footprint (none) -> Capacitor_SMD:C_0603_1608Metric; Rating (none) -> 50V X7R
- C33: value 22uF -> 1uF; footprint (none) -> Capacitor_SMD:C_0603_1608Metric; Rating (none) -> 16V X7R
- C34: value 100nF -> 47nF; footprint (none) -> Capacitor_SMD:C_0603_1608Metric; Rating (none) -> 25V X7R
- C38, C39: footprint (none) -> Capacitor_SMD:C_1206_3216Metric; Rating (none) -> 16V X7R
- C4, C6: footprint (none) -> Capacitor_SMD:C_0603_1608Metric; Rating (none) -> 50V C0G
- C40: value 22uF -> 47nF; footprint (none) -> Capacitor_SMD:C_0603_1608Metric; Rating (none) -> 50V X7R
- C41: value 47nF -> 22uF; footprint (none) -> Capacitor_SMD:C_1206_3216Metric; Rating (none) -> 16V X7R
- C42: value 4.7uF -> 22uF; footprint (none) -> Capacitor_SMD:C_1206_3216Metric; Rating (none) -> 16V X7R
- C43: footprint (none) -> Capacitor_SMD:C_0805_2012Metric; Rating (none) -> 100V X7R
- C44: value 1uF -> 10uF; footprint (none) -> Capacitor_SMD:C_0805_2012Metric; Rating (none) -> 16V X7R
- C45: value 100nF -> 220nF; footprint (none) -> Capacitor_SMD:C_0603_1608Metric; Rating (none) -> 16V X7R
- C46: value 10nF -> 1uF; footprint (none) -> Capacitor_SMD:C_0603_1608Metric; Rating (none) -> 16V X7R
- C47: value 10nF -> 100nF; footprint (none) -> Capacitor_SMD:C_0603_1608Metric; Rating (none) -> 50V X7R
- C48: value 1nF -> 100nF; footprint (none) -> Capacitor_SMD:C_0603_1608Metric; Rating (none) -> 16V X7R
- C49: value 4.7nF -> 100nF; footprint (none) -> Capacitor_SMD:C_0603_1608Metric; Rating (none) -> 16V X7R
- C5: value 10nF -> 100nF; footprint (none) -> Capacitor_SMD:C_0603_1608Metric; Rating (none) -> 16V X7R
- C51: value 220nF -> 22uF; footprint (none) -> Capacitor_SMD:C_1206_3216Metric; Rating (none) -> 10V X7R
- C52: value 100nF -> 22uF; footprint (none) -> Capacitor_SMD:C_1206_3216Metric; Rating (none) -> 10V X7R
- C8: value 1uF -> 10uF; footprint (none) -> Capacitor_SMD:C_0805_2012Metric; Rating (none) -> 10V X7R
- C82: value 100nF -> 10uF; footprint (none) -> Capacitor_SMD:C_1206_3216Metric; Rating (none) -> 16V X7R
- C9: value 47nF -> 1uF; footprint (none) -> Capacitor_SMD:C_0603_1608Metric; Rating (none) -> 16V X7R
- D13, D14: value ESD5Zxx -> ESD5Z6.0T1G
- D17, D18, D39, D7: value ESD5Zxx -> ESD5Z3.3T1G
- L1: value 8.2uH, 14mΩ -> 8.2uH; footprint (none) -> Inductor_SMD:L_Coilcraft_XAL1010-XXX; MPN (none) -> Coilcraft XAL1010-822MED (12.9 mOhm max, Isat 18.3 A) - Can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
- L2: value 6.8uH, 14mΩ -> 6.8uH; footprint (none) -> Inductor_SMD:L_Coilcraft_XAL7070-XXX; MPN (none) -> Coilcraft XAL7070-682MEC (19.6 mOhm max, Isat 12.8 A) - Can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
- R119, R120, R121: value 0 -> 100; footprint (none) -> Resistor_SMD:R_0603_1608Metric
- R12: value 4.7K -> 100K; footprint (none) -> Resistor_SMD:R_0603_1608Metric
- R122, R123, R124: value 0 -> 100K; footprint (none) -> Resistor_SMD:R_0603_1608Metric
- R13: value 4.7K -> 100; footprint (none) -> Resistor_SMD:R_0603_1608Metric
- R15: value 10 -> 5.1K; footprint (none) -> Resistor_SMD:R_0603_1608Metric
- R16: value 100K -> 10K; footprint (none) -> Resistor_SMD:R_0603_1608Metric
- R17: value 100K -> 10; footprint (none) -> Resistor_SMD:R_0603_1608Metric
- R18: value 24.9K -> 100K; footprint (none) -> Resistor_SMD:R_0603_1608Metric
- R19: value 5.1K -> 100K; footprint (none) -> Resistor_SMD:R_0603_1608Metric
- R2: value R_45deg -> LoadCell arm; now left out of the parts list
- R20, R21, R30, R66, R75, R83, R89, R90: footprint (none) -> Resistor_SMD:R_0603_1608Metric
- R22: value 6.04K -> 47; footprint (none) -> Resistor_SMD:R_0603_1608Metric
- R23: value 243K -> 5.1K; footprint (none) -> Resistor_SMD:R_0603_1608Metric
- R26: value 115K -> 1K; footprint (none) -> Resistor_SMD:R_0603_1608Metric; Tolerance (none) -> 1%
- R27: value 4.99K -> 100K; footprint (none) -> Resistor_SMD:R_0603_1608Metric; Tolerance (none) -> 1%
- R28: value 4.7K -> 8.2K; footprint (none) -> Resistor_SMD:R_0603_1608Metric; Tolerance (none) -> 1%
- R29, R31, R80: value 4.7K -> 10K; footprint (none) -> Resistor_SMD:R_0603_1608Metric
- R32: value 4.7K -> 1K; footprint (none) -> Resistor_SMD:R_0603_1608Metric; Tolerance (none) -> 1%
- R33: value 4.7K -> 100K; footprint (none) -> Resistor_SMD:R_0603_1608Metric; Tolerance (none) -> 1%
- R34: value 4.7K -> 5.6K; footprint (none) -> Resistor_SMD:R_0603_1608Metric; Tolerance (none) -> 1%
- R35: value 100K -> 1K; footprint (none) -> Resistor_SMD:R_0603_1608Metric
- R36: value 5.1K -> 1K; footprint (none) -> Resistor_SMD:R_0603_1608Metric
- R37, R39, R54: value 10K -> 1K; footprint (none) -> Resistor_SMD:R_0603_1608Metric
- R38: value 10K -> 1K; footprint (none) -> Resistor_SMD:R_0603_1608Metric; Tolerance (none) -> 1%
- R40: value 47 -> 4.7K; footprint (none) -> Resistor_SMD:R_0603_1608Metric
- R41: value 10K -> 1.2K; footprint (none) -> Resistor_SMD:R_0603_1608Metric; Tolerance (none) -> 1%
- R42: value 10K -> 4.7K; footprint (none) -> Resistor_SMD:R_0603_1608Metric
- R43: value 0 -> 820; footprint (none) -> Resistor_SMD:R_0603_1608Metric; Tolerance (none) -> 1%
- R44: value 10K -> 100K; footprint (none) -> Resistor_SMD:R_0603_1608Metric
- R45: value 100 -> 4.87K; footprint (none) -> Resistor_SMD:R_0603_1608Metric; Tolerance (none) -> 1%
- R46: value 100 -> 22K; footprint (none) -> Resistor_SMD:R_0603_1608Metric
- R50: value 43.2K -> 0; footprint (none) -> Resistor_SMD:R_0603_1608Metric; now not fitted
- R51: value 100 -> 4.7K; footprint (none) -> Resistor_SMD:R_0603_1608Metric
- R52: value 1K -> 2.2K; footprint (none) -> Resistor_SMD:R_0603_1608Metric
- R53: value 1M -> 2.2K; footprint (none) -> Resistor_SMD:R_0603_1608Metric
- R55: value 100K -> 22K; footprint (none) -> Resistor_SMD:R_0603_1608Metric
- R56: value 4.87K -> 22K; footprint (none) -> Resistor_SMD:R_0603_1608Metric
- R57: value 1.2K -> 0; footprint (none) -> Resistor_SMD:R_0603_1608Metric; now not fitted
- R58: value 820 -> 0; footprint (none) -> Resistor_SMD:R_0603_1608Metric; now not fitted
- R59: value 4.7K -> 243K; footprint (none) -> Resistor_SMD:R_0603_1608Metric; Tolerance (none) -> 1%
- R60: value 4.7K -> 6.04K; footprint (none) -> Resistor_SMD:R_0603_1608Metric; Tolerance (none) -> 1%
- R61: value 100K -> 10K; footprint (none) -> Resistor_SMD:R_0603_1608Metric; Tolerance (none) -> 1%
- R72: value 100K -> 0; footprint (none) -> Resistor_SMD:R_0603_1608Metric; now not fitted
- R76: value 100K -> 2.2K; footprint (none) -> Resistor_SMD:R_0603_1608Metric
- R77: value 10K -> 2.2K; footprint (none) -> Resistor_SMD:R_0603_1608Metric
- R78: footprint (none) -> Resistor_SMD:R_0603_1608Metric; Tolerance (none) -> 1%
- R79: value 100K -> 24.9K; footprint (none) -> Resistor_SMD:R_0603_1608Metric; Tolerance (none) -> 1%
- R81: value 100K -> 100; footprint (none) -> Resistor_SMD:R_0603_1608Metric
- R82: value 5.6K -> 10K; footprint (none) -> Resistor_SMD:R_0603_1608Metric
- R84: value 8.2K -> 4.7K; footprint (none) -> Resistor_SMD:R_0603_1608Metric
- R85: value 1K -> 4.7K; footprint (none) -> Resistor_SMD:R_0603_1608Metric
- R91, R92: value 10K -> 10; footprint (none) -> Resistor_SMD:R_0603_1608Metric
- R93: value 10K -> 100K; footprint (none) -> Resistor_SMD:R_0603_1608Metric; Tolerance (none) -> 1%
- SW1: value SW_Push -> RESET (optional); footprint (none) -> Button_Switch_SMD:SW_SPST_TL3342
- SW2: value SW_Push -> BOOT/SETUP (optional); footprint (none) -> Button_Switch_SMD:SW_SPST_TL3342
Connections:
- net TCA9548A SCX <3 is gone; now on net VALVE_IMON: R32.2
- net TCA9548A SDX <3 is gone; now on net OW_F1: R31.2
- net +24V: now also C23.2, C24.2, C29.2, C31.2, C32.2, R75.2, C36.1, D16.1 (K), J14.12 (+24V), J14.6 (+24V), J15.12 (+24V), J15.6 (+24V), J4.12 (+24V), J4.6 (+24V), R70.4 (F2), R73.2, U10.2 (VIN), U11.8 (VBUS), U4.10 (IN), U4.8 (IN), U4.9 (IN); no longer C13.2, C14.2, C42.2, C49.2, C50.2, R23.2, R26.2, R52.2, R55.2
- net +3V3: now also C14.1, C15.1, C48.1, C50.2, C51.2, C52.2, R17.2, R29.1, R30.1, R42.1, R46.1, R51.2, R55.1, R56.1, R66.2, R82.1, R84.2, R85.2, R90.2, R93.2, C1.1, C3.1, C53.2, C54.2, Q7.1 (G), Q8.1 (G), Q9.1 (G), R3.1, R4.1, R47.1, R68.1, R69.1, R88.1, R9.1, U11.6 (VS), U12.1 (A0), U12.2 (A1), U12.21 (A2), U12.24 (VCC), U3.15 (DVDD), U6.2 (3V3); no longer C31.1, C33.2, C38.2, C39.2, C40.2, C43.2, C44.1, C45.1, R12.1, R13.1, R15.2, R20.2, R28.2, R29.2, R30.2, R32.1, R33.1, R34.1, R37.1, R38.1, R41.2, R44.1, R54.2, R59.1, R77.1, R90.1, R91.1, R92.1, R93.1
- net +5V: now also C17.1, C35.2, C38.2, C39.2, C41.2, C42.2, C44.2, C45.2, R36.1, R37.1, R52.1, R53.1, R76.1, R77.1, R78.2, R83.1, C26.2, C28.2, C84.2, D16.2 (A), D37.1 (VDD), D38.1 (VDD), D4.1 (VDD), IC1.14 (VCC), J14.7 (+5V), J15.7 (+5V), J4.7 (+5V), PS1.2 (VIN), R64.1, R65.1, U5.8 (VCC), U7.8 (VCC), U9.8 (VCC); no longer C17.2, C18.2, C19.2, C20.2, C32.2, C52.1, R17.2
- net 1-Wire_1: now also R37.2, D22.1 (K), J4.8 (1-WIRE), Q9.3 (D); no longer R89.2
- net 1-Wire_2: now also R35.2, D41.1 (K), J14.8 (1-WIRE), Q7.3 (D); no longer R91.2
- net 1-Wire_3: now also R36.2, D44.1 (K), J15.8 (1-WIRE), Q8.3 (D); no longer D18.1 (K), R93.2
- net 1Y_out: now also R22.2, D4.4 (DIN); no longer D7.1 (K), R40.2
- net Boot: now also C13.1, R16.1, TP1.1, U6.27 (IO0); no longer C9.1, R41.1
- net EN: now also C2.1, PS1.4 (PG), R3.2, U6.3 (EN); no longer C8.1, R42.2
- net EN_PS2: now also R75.1, U10.3 (EN), U8.14 (ENOUT); no longer R55.1
- net EXP: now also C13.2, C14.2, C16.2, C17.2, C18.2, C20.2, C23.1, C24.1, C29.1, C31.1, C33.2, C34.2, C35.1, C40.2, C41.1, C43.2, C44.1, C45.1, C46.1, C48.2, C52.1, R12.2, R122.1, R123.1, R124.1, R15.2, R18.2, R2.1, R20.2, R23.2, R28.2, R34.1, R41.2, R44.2, R45.1, R61.1, R79.1, C1.2, C10.2, C2.2, C25.1, C26.1, C27.2, C28.1, C3.2, C30.2, C36.2, C53.1, C54.1, C79.2, C80.2, C81.2, C84.1, D1.2 (A), D19.2 (A), D2.2 (A), D20.2 (A), D22.2 (A), D23.2, D37.3 (VSS), D38.3 (VSS), D4.3 (VSS), D40.2 (A), D41.2 (A), D42.2 (A), D43.2 (A), D44.2 (A), D8.2 (A), D9.2 (A), IC1.1 (1~{OE}), IC1.10 (3~{OE}), IC1.12 (4A), IC1.13 (4~{OE}), IC1.7 (GND), IC1.9 (3A), J1.A1/B12 (GND_A), J1.B1/A12 (GND_B), J1.SH1 (SHIELD), J1.SH2 (SHIELD), J1.SH3 (SHIELD), J1.SH4 (SHIELD), J11.2 (E-), J11.5 (SH), J13.2 (Pin_2), J14.10 (GND), J14.11 (GND), J14.5 (GND), J14.9 (GND), J15.10 (GND), J15.11 (GND), J15.5 (GND), J15.9 (GND), J4.10 (GND), J4.11 (GND), J4.5 (GND), J4.9 (GND), J5.2, J5.3, J5.S1 (SHIELD), PS1.1 (PGND), PS1.9 (EP), Q1.2 (S), Q18.2 (S), Q19.2 (S), Q2.2 (S), Q20.2 (S), Q3.2 (S), Q4.2 (S), Q5.2 (S), Q6.2 (S), R10.2, R11.2, R48.1, R74.1, R8.1, R94.1, U1.2, U10.1 (PGND), U10.9 (AGND), U11.1 (A1), U11.2 (A0), U11.7 (GND), U12.12 (GND), U2.3 (GND), U3.10 (XIN), U3.7 (REFN), U3.8 (AVSS), U3.9 (DVSS), U4.15 (EXP), U4.16 (EXP), U4.17 (EXP), U4.18 (EXP), U4.19 (EXP), U4.2 (GND), U4.20 (EXP), U4.21 (EXP), U5.4 (GND), U6.1 (GND), U6.40 (GND), U6.41_1 (GND), U6.41_2 (GND), U6.41_3 (GND), U6.41_4 (GND), U6.41_5 (GND), U6.41_6 (GND), U6.41_7 (GND), U6.41_8 (GND), U6.41_9 (GND), U7.4 (GND), U8.12 (GND), U9.4 (GND); no longer C13.1, C14.1, C17.1, C18.1, C20.1, C23.2, C29.2, C31.2, C33.1, C35.2, C37.2, C40.1, C41.2, C43.1, C44.2, C45.2, C46.2, C47.2, C48.1, C49.1, C52.2, C7.2, R18.1, R27.1, R36.2, R39.1, R50.1, R56.1, R57.2, R61.2, R66.2, R72.2, R75.2, R76.2, R78.2, R79.2, R82.1, R84.2
- net HGATE: now also R81.1, D21.2 (A), R67.1, U8.6 (HGATE), Z1.1 (K); no longer R51.1
- net IN+: now also R91.2, R70.2 (S1), U8.2 (SENSE)
- net LEAK_BASE: now also U6.7 (IO7)
- net LEAK_EXC: now also U6.22 (IO14)
- net LOADCELL_DRDY: now also U3.12 (DRDY), U6.8 (IO15)
- net MUX_RST_N: now also R90.1, U12.3 (~{RESET}), U6.23 (IO21); no longer R30.1
- net OE_1: now also D18.1 (K), J4.1 (OE)
- net OE_2: now also D40.1 (K), J14.1 (OE); no longer D14.1 (K)
- net OE_3: now also D43.1 (K), J15.1 (OE); no longer D17.1 (K)
- net OE_DRV: now also U6.26 (IO45); no longer R75.1, R76.1, R79.1
- net OW_F1: now also Q9.2 (S), U6.19 (IO11); no longer R77.2
- net OW_F2: now also R29.2, Q7.2 (S), U6.20 (IO12); no longer R90.2
- net OW_F3: now also R30.2, Q8.2 (S), U6.21 (IO13); no longer R92.2
- net PG_5V: now also R66.1, U10.4 (PG), U6.33 (IO40); no longer R16.1
- net PUMP_EN: now also IC1.5 (2A), U6.34 (IO41)
- net PWR_ALERT_N: now also R82.2, U11.3 (ALERT), U6.11 (IO18); no longer R44.2
- net RING_DATA: now also R21.2, IC1.2 (1A), U6.12 (IO8); no longer R39.2
- net RXD0: now also U6.36 (RXD0)
- net SCL_0: now also R85.1, U12.22 (SCL), U6.25 (IO48); no longer R29.1
- net SCL_1: now also R4.2, U11.5 (SCL), U2.1 (SCL), U3.13 (SCLK), U6.10 (IO17); no longer R12.2, R34.2
- net SCL_F1: now also R50.2, R52.2, D8.1 (K), J4.3 (SCL), U5.5 (TY), U5.6 (RY); no longer R120.2
- net SCL_F2: now also D13.1 (K), R58.2, J14.3 (SCL), R64.2, U7.5 (TY), U7.6 (RY); no longer R122.2
- net SCL_F3: now also R72.2, R76.2, D19.1 (K), J15.3 (SCL), U9.5 (TY), U9.6 (RY); no longer R124.2
- net SC_0: now also R46.2, R50.1, U12.5 (SC0), U5.7 (SY); no longer R120.1
- net SC_1: now also R55.2, R58.1, U12.7 (SC1), U7.7 (SY); no longer R122.1
- net SC_2: now also R72.1, R68.2, U12.9 (SC2), U9.7 (SY); no longer R124.1
- net SDA_0: now also R84.1, U12.23 (SDA), U6.24 (IO47); no longer R28.1
- net SDA_1: now also R9.2, U11.4 (SDA), U2.4 (SDA), U3.14 (SDIO), U6.9 (IO16); no longer R13.2, R33.2
- net SDA_F1: now also R53.2, D9.1 (K), J4.4 (SDA), R49.1, U5.2 (RX), U5.3 (TX); no longer R119.1
- net SDA_F2: now also D14.1 (K), R57.1, J14.4 (SDA), R65.2, U7.2 (RX), U7.3 (TX); no longer R121.1
- net SDA_F3: now also R77.2, D20.1 (K), J15.4 (SDA), R71.1, U9.2 (RX), U9.3 (TX); no longer D39.1 (K), R123.1
- net SD_0: now also R47.2, R49.2, U12.4 (SD0), U5.1 (SX); no longer R119.2
- net SD_1: now also R56.2, R57.2, U12.6 (SD1), U7.1 (SX); no longer R121.2
- net SD_2: now also R69.2, R71.2, U12.8 (SD2), U9.1 (SX); no longer R123.2
- net TANK_LOW: now also R54.2, C27.1, IC1.4 (2~{OE}), U6.35 (IO42)
- net TCA9548A SCX >2: now also R89.2, U12.11 (SC3), U12.14 (SC4), U12.16 (SC5), U12.18 (SC6), U12.20 (SC7); no longer R38.2
- net TCA9548A SDX >2: now also R88.2, U12.10 (SD3), U12.13 (SD4), U12.15 (SD5), U12.17 (SD6), U12.19 (SD7); no longer R37.2
- net TXD0: now also U6.37 (TXD0)
- net USB_D+: now also R5.1, U6.14 (IO20); no longer R43.1
- net USB_D-: now also R6.1, U6.13 (IO19)
- net V24_SENSE: now also C20.1, R38.1, U6.4 (IO4); no longer C4.1, R81.2, R85.1
- net VALVE_IMON: now also C18.1, U6.5 (IO5); no longer C48.2, C6.1
- net VALVE_RAIL: now also R27.1, C25.2, C79.1, C80.1, C81.1, D34.1 (K), D35.1 (K), D36.1 (K), J10.1, J8.1, J9.1, R48.2, U4.5 (OUT), U4.6 (OUT), U4.7 (OUT); no longer C51.2, R83.1
- net VALVE_RAIL_EN: now also R40.1, U6.31 (IO38); no longer R60.1
- net VALVE_RAIL_SENSE_DIV: now also C16.1, R26.2, U6.6 (IO6); no longer C5.1
- net VIN_FLT_N: now also R80.1, U6.32 (IO39), U8.13 (*FLT); no longer R54.1
- net nRESET_1: now also D17.1 (K), J4.2 (nRESET)
- net nRESET_2: now also D39.1 (K), J14.2 (nRESET); no longer D13.1 (K)
- net nRESET_3: now also D42.1 (K), J15.2 (nRESET)
- net nRESET_DRV: now also U6.16 (IO46); no longer R66.1, R72.1, R78.1
- net at R60.2: now also R59.1, U8.10 (UV); no longer R61.1
- net at R22.1: now also IC1.3 (1Y); no longer R21.2
- net S+: now reaches R2.2
- net S+: now also R13.1, D1.1 (K), J11.3 (S+), R1.1; no longer R45.1
- net at R43.2: now also U4.14 (IMON)
- net U2_VDD: now reaches R17.1
- net U2_VDD: now also C12.1, C8.1, U2.2 (VDD); no longer R18.2
- net VIN: now reaches R59.2
- net VIN: now also C43.1, R33.2, D23.1, J5.1, J5.4, Q10.2, R63.2
- net at R23.1: now also J1.B5 (CC2); no longer R22.2
- net at R26.1, R27.2: now also R28.1
- net at C37.1: now also L1.1, U10.8 (SW); no longer R2.1
- net NRST_G3: now reaches R20.1
- net NRST_G3: now also Q6.1 (G); no longer R50.2
- net at R15.1: now also J1.A5 (CC1); no longer C12.1
- net at R83.2: now also PS1.3 (EN); no longer R84.1
- net at L2.1: now also C49.1, PS1.8 (SW); no longer C24.1
- net NRST_G2: now reaches R19.1
- net NRST_G2: now also Q5.1 (G)
- net 3V3: no longer names the net of C7.1
- net 3V3: now also C6.1, R14.2, U3.2 (VIN1N); no longer R42.1
- new net: Q18.1 (G), R119.2, R122.2
- new net: Q10.3, Q11.1 (S_1), Q11.2 (S_2), Q11.3 (S_3), U8.5 (SOURCE), Z1.2 (A), Z2.2 (A)
- new net: Q11.4 (G), U8.4 (DGATE), Z2.1 (K)
- new net: R33.1, R34.2, R38.2
- new net: C47.1, R91.1, U11.10 (IN+)
- new net: C47.2, R92.1, U11.9 (IN-)
- new net: Q19.1 (G), R120.2, R123.2
- new net: C49.2, PS1.7 (BOOT)
- new net: C37.2, U10.7 (BOOT)
- new net: D35.2 (A), J9.2, Q19.3 (D)
- new net: D7.1 (K), J13.1 (Pin_1), R51.1, R54.1
- new net: C4.1, C7.2, R13.2, U3.3 (VIN1P)
- new net: C10.1, U3.6 (VBG)
- new net: R73.1, R74.2, U8.16 (FB)
- new net: D36.2 (A), J10.2, Q20.3 (D)
- new net: D34.2 (A), J8.2, Q18.3 (D)
- new net: R78.1, R79.2, U10.5 (FB)
- new net: C33.1, U10.6 (VCC)
- new net: C11.1, U3.4 (VIN2N)
- new net: C11.2, U3.5 (VIN2P)
- new net: C34.1, U8.15 (TMR)
- new net: Q20.1 (G), R121.2, R124.2
- new net: R5.2, U1.4
- new net: C40.1, D21.1 (K), R81.2
- new net: R39.2, R41.1, R43.1
- new net: R62.1, U8.9 (*SHDN)
- new net: R60.1, R61.2, U8.11 (OV)
- new net: D37.2 (DOUT), D38.4 (DIN)
- new net: D37.4 (DIN), D4.2 (DOUT)
- new net: R40.2, R44.1, U4.3 (EN)
- new net: Q10.1, R67.2
- new net: R6.2, U1.6
- new net: R42.2, U4.12 (DIAG_EN)
- new net: PS1.5 (FB), R93.1, R94.2
- new net: C46.2, PS1.6 (VCC)
- new net: R45.2, U4.13 (ILIM)
- new net DOSE_SEL0: U6.18 (IO10)
- new net DOSE_SEL1: U6.15 (IO3)
- new net E+: C5.1, C9.1, J11.1 (E+), R1.2, R7.1, U3.1 (REFP), U3.16 (AVDD/LDO)
- new net IN-: R70.3 (S2), R92.2, U8.1 (OUT)
- new net LED_DOUT: D38.2 (DOUT)
- new net M2_DRAIN: Q11.10 (D_6), Q11.11 (D_7), Q11.5 (D_1), Q11.6 (D_2), Q11.7 (D_3), Q11.8 (D_4), Q11.9 (D_5), R70.1 (F1)
- new net NRST_G1: Q4.1 (G), R18.1
- new net OE_1_D: Q1.3 (D)
- new net OE_2_D: Q2.3 (D)
- new net OE_3_D: Q3.3 (D)
- new net OE_G1: Q1.1 (G), R10.1
- new net OE_G2: Q2.1 (G), R11.1
- new net OE_G3: Q3.1 (G), R12.1
- new net PUMP_GDRV: IC1.6 (2Y)
- new net S-: D2.1 (K), J11.4 (S-), R14.1, R7.2, R8.2
- new net U8_VCC: C30.1, R62.2, R63.1, U8.8 (VCC)
- new net USB_C_DN: J1.A7 (DN1), J1.B7 (DN2), U1.1
- new net USB_C_DP: J1.A6 (DP1), J1.B6 (DP2), U1.3
- new net USB_VBUS: J1.A4/B9 (VBUS_A), J1.B4/AP (VBUS_B), U1.5
- new net VALVE_IMON_DIV: C19.2, R32.1, R39.1
- new net Valve_0: R119.1, U6.39 (IO1)
- new net Valve_1: R120.1, U6.38 (IO2)
- new net Valve_2: R121.1, U6.17 (IO9)
- new net nRESET_1_D: Q4.3 (D)
- new net nRESET_2_D: Q5.3 (D)
- new net nRESET_3_D: Q6.3 (D)
- no-connect marks 27 -> 10
Other:
- removed sheet Basic_Floor_PCB
- added sheet Base_IO (Base_IO.kicad_sch)
- note added: "0R links: plain-I2C build only - DNP while U5/U7/U9 are fitted"
- note added: "ESD per line: Z6.0 = 5 V Z3.3 = 3.3 V"
- note added: "Floor Cables"
- note added: "Floor boards (x3): separate KiCad project GrowHub_Floor (2-layer)."
- note added: "I2C Buffer"
- note added: "Load Cell 30KG"
- note added: "MCU"
- note added: "Valve Driver"
- note removed: "E+"
- note removed: "E-"
- note removed: "Floor cabling needs revision"
- note removed: "In reality 3 "Basic Floor" will be printed"
- note removed: "Load Cell"
- note removed: "Out of PCB"
- note removed: "S+"
- note removed: "S-"
- note removed: "TCA9548A Pull-up Out 0-2"
